File: 300BaudModem.kicad_pcb (KiCad board)
At the start: 4 copper layers, 160 x 100 mm, 27 parts, among them U1 LM7905, X2 Raw

Commit message: updates
Parts:
- added REF**: Relay_DPDT_Panasonic_JW2, Relays_THT:Relay_DPDT_Panasonic_JW2, F.Cu at (118.4, 68.3)
Other:
- board text added: "IN DEVELOPMENT"

Commit message: updates
Parts:
- removed DB_9M: JP***, conn_dsub:DB_9M
- added DB_9F: JP***, conn_dsub:DB_9F, F.Cu at (79.2, 117.9)
- moved REF** 45.2 mm to (151.6, 103.9)
- moved REF** 1.02 mm to (82.3, 68.6)
- moved REF** 1.02 mm to (82.3, 63.5)
- moved REF** 1.02 mm to (79.8, 68.6)
- moved REF** 1.02 mm to (79.8, 63.5)
- moved REF** 1.02 mm to (84.8, 68.6)
- moved REF** 1.02 mm to (84.8, 63.5)
Other:
- board text added: "DCE"
- board text added: "DTE"
