File: 300BaudModem.kicad_pcb (KiCad board)
At the start: 4 copper layers, 160 x 100 mm, 28 parts, among them U1 LM7905, X2 Raw

Commit message: updates
Parts:
- removed the REF** at (118.4, 68.3)
- REF**: value RJ12_E -> RJ45_8; footprint Connectors:RJ12_E -> Connectors:RJ45_8
- REF**: value PinHeader_1x3_P2.54_Drill1.1mm -> Pin_Header_Straight_1x08_Pitch2.54mm; footprint Digikey:PinHeader_1x3_P2.54_Drill1.1mm -> Pin_Headers:Pin_Header_Straight_1x08_Pitch2.54mm
- moved REF** 6.86 mm to (104.1, 102.1), turned to 180 degrees
- moved REF** 4.66 mm to (88.4, 88.6)
- moved REF** 4.28 mm to (96.3, 84.8)
Other:
- board text added: "TEL INTERFACE SLIC E&M"
- board text removed: "SLIC X100M"

Commit message: updates
Parts:
- removed the REF** at (74.9, 142.2)
- removed the REF** at (210.2, 104.1)
- added REF**: MountingHole_2.5mm_Pad_Via, Mounting_Holes:MountingHole_2.5mm_Pad_Via, F.Cu at (78.6, 47.8)
- added REF**: MountingHole_2.5mm_Pad_Via, Mounting_Holes:MountingHole_2.5mm_Pad_Via, F.Cu at (78.4, 136.7)
- moved REF** 36.1 mm to (169.0, 67.6), turned to 270 degrees
- moved REF** 29.9 mm to (181.1, 64.1)
- moved REF** 17.6 mm to (160.5, 88.6)
- moved REF** 13.4 mm to (137.2, 82.0)
Other:
- board text removed: "16550 to Backplane"

Commit message: updates
Parts:
- removed the REF** at (181.1, 64.1)
- removed the REF** at (93.3, 73.0)
- removed the REF** at (199.1, 47.0)
- added REF**: Pin_Header_Straight_1x08_Pitch2.54mm, Pin_Headers:Pin_Header_Straight_1x08_Pitch2.54mm, F.Cu at (95.2, 81.9)
- added REF**: Fuse_0679H, Fuse_Holders_and_Fuses:Fuse_0679H, F.Cu at (216.5, 52.7)
- added REF**: Pin_Header_Straight_1x08_Pitch2.54mm, Pin_Headers:Pin_Header_Straight_1x08_Pitch2.54mm, F.Cu at (106.0, 85.4)
- added REF**: Pin_Header_Straight_2x10_Pitch2.54mm, Pin_Headers:Pin_Header_Straight_2x10_Pitch2.54mm, F.Cu at (139.1, 65.3)
- added X2: Raw, Sebs:mj-2135-MJ-2135, F.Cu at (80.6, 67.9)
- moved REF** 114.9 mm to (193.9, 56.0), turned to 90 degrees
- moved REF** 114.2 mm to (193.9, 61.1), turned to 90 degrees
- moved REF** 109.8 mm to (191.4, 56.0), turned to 90 degrees
- moved REF** 109.1 mm to (191.4, 61.1), turned to 90 degrees
- moved REF** 104.8 mm to (188.8, 56.0), turned to 90 degrees
- moved REF** 104.0 mm to (188.8, 61.1), turned to 90 degrees
- moved REF** 95.4 mm to (170.8, 58.4)
- moved REF** 56.8 mm to (173.3, 73.2), turned to 0 degrees
- moved REF** 37.3 mm to (132.1, 132.1), turned to 180 degrees
- moved REF** 32.7 mm to (154.3, 56.5)
- moved REF** 19.0 mm to (99.7, 103.5)
- moved REF** 18.2 mm to (150.9, 128.3)
- moved REF** 16.5 mm to (153.7, 73.7), turned to 0 degrees
- moved REF** 13.9 mm to (106.1, 115.9)
- moved REF** 13.9 mm to (139.2, 95.8)
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Other:
- board text added: "I/O Interface to 2 x TRRS"
- board text added: "I/O Interface to RJ45"
- board text removed: "Serial to WIFI Modem"
- board text removed: "TEL INTERFACE SLIC E&M"

Commit message: general updates
Parts:
- removed the REF** at (95.2, 81.9)
- added REF**: LED_D3.0mm, LEDs:LED_D3.0mm, F.Cu at (241.3, 106.7)
- added REF**: LED_D3.0mm, LEDs:LED_D3.0mm, F.Cu at (241.3, 114.3)
- added REF**: LED_D3.0mm, LEDs:LED_D3.0mm, F.Cu at (241.3, 121.9)
- added REF**: LED_D3.0mm, LEDs:LED_D3.0mm, F.Cu at (241.3, 129.5)
- added REF**: LED_D3.0mm, LEDs:LED_D3.0mm, F.Cu at (241.3, 91.4)
- added REF**: MountingHole_2.5mm_Pad_Via, Mounting_Holes:MountingHole_2.5mm_Pad_Via, F.Cu at (241.3, 47.8)
- added REF**: MountingHole_2.5mm_Pad_Via, Mounting_Holes:MountingHole_2.5mm_Pad_Via, F.Cu at (241.3, 136.7)
- added REF**: Pin_Header_Straight_2x05_Pitch2.54mm, Pin_Headers:Pin_Header_Straight_2x05_Pitch2.54mm, F.Cu at (192.4, 66.0)
- added REF**: Pin_Header_Straight_2x05_Pitch2.54mm, Pin_Headers:Pin_Header_Straight_2x05_Pitch2.54mm, F.Cu at (240.0, 64.8)
- added REF**: LED_D3.0mm, LEDs:LED_D3.0mm, F.Cu at (241.3, 58.4)
- added REF**: LED_D3.0mm, LEDs:LED_D3.0mm, F.Cu at (241.3, 83.8)
- added REF**: LED_D3.0mm, LEDs:LED_D3.0mm, F.Cu at (241.3, 99.1)
- REF**: footprint Mechanical_Sockets:Socket_DIN41612-CaseC1-full-Male-96Pin-3rows -> Sebs:Socket_DIN41612-CaseC1-full-Male-96Pin-3rows
- moved REF** 18.5 mm to (97.8, 85.1)
Other:
- board size 160 x 100 mm -> 172.7 x 100 mm
- board text added: "AUX1"
- board text added: "AUX2"
- board text added: "CD"
- board text added: "OH"
- board text added: "PWR"
- board text added: "RI"
- board text added: "RX"
- board text added: "TX"
- board text added: "vScore Front Pannel Breakoff"
- board text removed: "LEDS: TX,RX,CD,OH,RI, PWR"

Commit message: io interface updates
Parts:
- moved REF** 25.1 mm to (215.9, 57.1)
- moved REF** 17.8 mm to (241.3, 76.2)
- moved REF** 9.53 mm to (207.0, 52.7)
- moved REF** 7.62 mm to (240.0, 57.1)
- moved X2 0.64 mm to (80.6, 68.6)
- moved X2 0.63 mm to (80.6, 78.7)
Other:
- board text added: "AA"
- board text added: "DSR"
- board text added: "DTR"
- board text added: "HEGARS 300 MODEM MAX"
- board text removed: "AUX1"
- board text removed: "AUX2"
- board text removed: "PWR"

Commit message: updates
Parts:
- moved REF** 1.27 mm to (87.6, 88.3)
Other:
- board text added: "HEGARS 300 MODEM nMAX"
- board text added: "Romani ite domum"
- board text removed: "HEGARS 300 MODEM MAX"
- board text removed: "IN DEVELOPMENT"
Changed lines of the file:
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@@
   )
   (module Connectors:RJ45_8 (layer F.Cu)
-    (at 88.9 88.265 270)
+    (at 87.63 88.265 270)
     (tags RJ45)
     (fp_text reference REF** (at 3.3 6.35 90) (layer F.SilkS)
@@
   )
   (gr_line (start 237.49 142.24) (end 237.49 42.291) (layer F.SilkS) (width 0.12))
-  (gr_text "HEGARS 300 MODEM MAX" (at 246.38 57.15 90) (layer F.SilkS)
+  (gr_text "HEGARS 300 MODEM nMAX" (at 246.38 57.15 90) (layer F.SilkS)
     (effects (font (size 1 1) (thickness 0.15)))
   )
@@
     (effects (font (size 1 1) (thickness 0.15)) (justify left))
   )
-  (gr_text "IN DEVELOPMENT" (at 151.892 47.498) (layer F.SilkS)
+  (gr_text "Romani ite domum" (at 154.94 48.26) (layer F.SilkS)
     (effects (font (size 3 3) (thickness 0.3)))
   )

Commit message: updates
Parts:
- moved REF** 10.6 mm to (217.2, 49.5)
- moved X2 0.64 mm to (81.3, 68.6)
- moved X2 0.64 mm to (81.3, 78.7)
- moved REF** 0.63 mm to (87.0, 88.3)
Other:
- board text added: "Aedificium - Romani ite domum"
- board text added: "vScore Front Pannel"
- board text removed: "Romani ite domum"
- board text removed: "vScore Front Pannel Breakoff"
Changed lines of the file:
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@@
   )
   (module Fuse_Holders_and_Fuses:Fuse_0679H (layer F.Cu)
-    (at 207.01 52.705)
+    (at 217.17 49.53)
     (descr "0679H Series, 2410 Size")
     (tags Fuse)
@@
   )
   (module Sebs:mj-2135-MJ-2135 (layer F.Cu)
-    (at 80.645 68.58 90)
+    (at 81.28 68.58 90)
     (attr virtual)
     (fp_text reference X2 (at 0 0 -90) (layer F.SilkS)
@@
   )
   (module Connectors:RJ45_8 (layer F.Cu)
-    (at 87.63 88.265 270)
+    (at 86.995 88.265 270)
     (tags RJ45)
     (fp_text reference REF** (at 3.3 6.35 90) (layer F.SilkS)
@@
   )
   (module Sebs:mj-2135-MJ-2135 (layer F.Cu)
-    (at 80.645 78.74 90)
+    (at 81.28 78.74 90)
     (attr virtual)
     (fp_text reference X2 (at 0 0 -90) (layer F.SilkS)
@@
     (effects (font (size 1 1) (thickness 0.15)))
   )
-  (gr_text "vScore Front Pannel Breakoff" (at 236.22 55.88 90) (layer F.SilkS)
+  (gr_text "vScore Front Pannel" (at 236.22 55.88 90) (layer F.SilkS)
     (effects (font (size 1 1) (thickness 0.15)))
   )
@@
     (effects (font (size 1 1) (thickness 0.15)) (justify left))
   )
-  (gr_text "Romani ite domum" (at 154.94 48.26) (layer F.SilkS)
+  (gr_text "Aedificium - Romani ite domum" (at 167.64 48.26) (layer F.SilkS)
     (effects (font (size 3 3) (thickness 0.3)))
   )
