File: 300BaudModem.kicad_pcb (KiCad board)
At the start: 4 copper layers, 172.7 x 100 mm, 40 parts, among them U1 LM7905, X2 Raw

Commit message: updates
Parts:
- removed the REF** at (241.3, 121.9)
- removed the REF** at (241.3, 129.5)
- added REF**: SW_TH_Tactile_Omron_B3F-10xx, Buttons_Switches_THT:SW_TH_Tactile_Omron_B3F-10xx, F.Cu at (244.6, 71.1)
- added REF**: LED_D3.0mm, LEDs:LED_D3.0mm, F.Cu at (241.3, 123.2)
- added REF**: LED_D3.0mm, LEDs:LED_D3.0mm, F.Cu at (241.3, 130.8)
- moved REF** 8.89 mm to (208.3, 49.3)
- moved REF** 4.02 mm to (217.2, 53.3)
- moved REF** 3.81 mm to (240.0, 53.3)
- moved REF** 1.27 mm to (241.3, 85.1)
- moved REF** 1.27 mm to (241.3, 100.3)
- moved REF** 1.27 mm to (241.3, 108.0)
- moved REF** 1.27 mm to (241.3, 115.6)
- moved REF** 1.27 mm to (241.3, 77.5)
- moved REF** 1.27 mm to (241.3, 92.7)
Changed lines of the file:
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@@
     (tracks 0)
     (zones 0)
-    (modules 40)
+    (modules 41)
     (nets 1)
   )
@@
     (uvia_drill 0.1)
   )
+  (module Buttons_Switches_THT:SW_TH_Tactile_Omron_B3F-10xx (layer F.Cu)
+    (at 244.602 71.12 180)
+    (descr SW_TH_Tactile_Omron_B3F-10xx_https://www.omron.com/ecb/products/pdf/en-b3f.pdf)
+    (tags "Omron B3F-10xx")
+    (fp_text reference REF** (at 3.25 -2.05) (layer F.SilkS)
+      (effects (font (size 1 1) (thickness 0.15)))
+    )
+    (fp_text value SW_TH_Tactile_Omron_B3F-10xx (at 3.2 6.5) (layer F.Fab)
+      (effects (font (size 1 1) (thickness 0.15)))
+    )
+    (fp_line (start 0.25 5.25) (end 6.25 5.25) (layer F.Fab) (width 0.1))
+    (fp_line (start 6.37 0.91) (end 6.37 3.59) (layer F.SilkS) (width 0.12))
+    (fp_line (start 0.13 3.59) (end 0.13 0.91) (layer F.SilkS) (width 0.12))
+    (fp_line (start 0.28 -0.87) (end 6.22 -0.87) (layer F.SilkS) (width 0.12))
+    (fp_line (start 0.28 5.37) (end 6.22 5.37) (layer F.SilkS) (width 0.12))
+    (fp_circle (center 3.25 2.25) (end 4.25 3.25) (layer F.SilkS) (width 0.12))
+    (fp_line (start -1.1 -1.15) (end -1.1 5.6) (layer F.CrtYd) (width 0.05))
+    (fp_line (start -1.1 5.6) (end 7.6 5.6) (layer F.CrtYd) (width 0.05))
+    (fp_line (start 7.6 5.6) (end 7.6 -1.1) (layer F.CrtYd) (width 0.05))
+    (fp_line (start 7.65 -1.15) (end -1.1 -1.15) (layer F.CrtYd) (width 0.05))
+    (fp_line (start 0.25 -0.75) (end 6.25 -0.75) (layer F.Fab) (width 0.1))
+    (fp_line (start 6.25 -0.75) (end 6.25 5.25) (layer F.Fab) (width 0.1))
+    (fp_line (start 0.25 -0.75) (end 0.25 5.25) (layer F.Fab) (width 0.1))
+    (fp_text user %R (at 3.25 2.25) (layer F.Fab)
+      (effects (font (size 1 1) (thickness 0.15)))
+    )
+    (pad 4 thru_hole circle (at 6.5 4.5 180) (size 1.7 1.7) (drill 1) (layers *.Cu *.Mask))
+    (pad 3 thru_hole circle (at 0 4.5 180) (size 1.7 1.7) (drill 1) (layers *.Cu *.Mask))
+    (pad 2 thru_hole circle (at 6.5 0 180) (size 1.7 1.7) (drill 1) (layers *.Cu *.Mask))
+    (pad 1 thru_hole circle (at 0 0 180) (size 1.7 1.7) (drill 1) (layers *.Cu *.Mask))
+    (model ${KISYS3DMOD}/Buttons_Switches_THT.3dshapes/SW_TH_Tactile_Omron_B3F-10xx.wrl
+      (at (xyz 0 0 0))
+      (scale (xyz 1 1 1))
+      (rotate (xyz 0 0 0))
+    )
+  )
   (module LEDs:LED_D3.0mm (layer F.Cu)
-    (at 241.3 76.2 90)
+    (at 241.3 77.47 90)
     (descr "LED, diameter 3.0mm, 2 pins")
     (tags "LED diameter 3.0mm 2 pins")
@@
   )
   (module LEDs:LED_D3.0mm (layer F.Cu)
-    (at 241.3 91.44 90)
+    (at 241.3 92.71 90)
     (descr "LED, diameter 3.0mm, 2 pins")
     (tags "LED diameter 3.0mm 2 pins")
@@
   )
   (module Pin_Headers:Pin_Header_Straight_2x05_Pitch2.54mm (layer F.Cu)
-    (at 215.9 57.15)
+    (at 217.17 53.34)
     (descr "Through hole straight pin header, 2x05, 2.54mm pitch, double rows")
     (tags "Through hole pin header THT 2x05 2.54mm double row")
@@
   )
   (module Pin_Headers:Pin_Header_Straight_2x05_Pitch2.54mm (layer F.Cu)
-    (at 240.03 57.15)
+    (at 240.03 53.34)
     (descr "Through hole straight pin header, 2x05, 2.54mm pitch, double rows")
     (tags "Through hole pin header THT 2x05 2.54mm double row")
@@
   )
   (module LEDs:LED_D3.0mm (layer F.Cu)
-    (at 241.3 83.82 90)
+    (at 241.3 85.09 90)
     (descr "LED, diameter 3.0mm, 2 pins")
     (tags "LED diameter 3.0mm 2 pins")
@@
   )
   (module LEDs:LED_D3.0mm (layer F.Cu)
-    (at 241.3 99.06 90)
+    (at 241.3 100.33 90)
     (descr "LED, diameter 3.0mm, 2 pins")
     (tags "LED diameter 3.0mm 2 pins")
@@
   )
   (module LEDs:LED_D3.0mm (layer F.Cu)
-    (at 241.3 106.68 90)
+    (at 241.3 107.95 90)
     (descr "LED, diameter 3.0mm, 2 pins")
     (tags "LED diameter 3.0mm 2 pins")
@@
   )
   (module LEDs:LED_D3.0mm (layer F.Cu)
-    (at 241.3 114.3 90)
+    (at 241.3 115.57 90)
     (descr "LED, diameter 3.0mm, 2 pins")
     (tags "LED diameter 3.0mm 2 pins")
@@
   )
   (module LEDs:LED_D3.0mm (layer F.Cu)
-    (at 241.3 121.92 90)
+    (at 241.3 123.19 90)
     (descr "LED, diameter 3.0mm, 2 pins")
     (tags "LED diameter 3.0mm 2 pins")
@@
   )
   (module LEDs:LED_D3.0mm (layer F.Cu)
-    (at 241.3 129.54 90)
+    (at 241.3 130.81 90)
     (descr "LED, diameter 3.0mm, 2 pins")
     (tags "LED diameter 3.0mm 2 pins")
@@
   )
   (module Fuse_Holders_and_Fuses:Fuse_0679H (layer F.Cu)
-    (at 217.17 49.53)
+    (at 208.28 49.276)
     (descr "0679H Series, 2410 Size")
     (tags Fuse)
@@
     (arrow2b (pts (xy 58.233403 136.608738) (xy 57.649398 135.48098)))
   )
-  (gr_line (start 237.49 142.24) (end 237.49 42.291) (layer F.SilkS) (width 0.12))
+  (gr_line (start 237.998 142.24) (end 237.998 42.291) (layer F.SilkS) (width 0.12))
   (gr_text "HEGARS 300 MODEM nMAX" (at 246.38 57.15 90) (layer F.SilkS)
     (effects (font (size 1 1) (thickness 0.15)))
   )
-  (gr_text DSR (at 246.38 74.93 90) (layer F.SilkS)
+  (gr_text DSR (at 246.38 76.2 90) (layer F.SilkS)
     (effects (font (size 1 1) (thickness 0.15)))
   )
-  (gr_line (start 234.95 71.12) (end 247.65 71.12) (layer F.SilkS) (width 0.12))
-  (gr_line (start 245.11 142.24) (end 245.11 42.291) (layer F.SilkS) (width 0.12))
-  (gr_line (start 234.95 78.74) (end 247.65 78.74) (layer F.SilkS) (width 0.12))
-  (gr_line (start 234.95 86.36) (end 247.65 86.36) (layer F.SilkS) (width 0.12))
-  (gr_line (start 234.95 93.98) (end 247.65 93.98) (layer F.SilkS) (width 0.12))
-  (gr_line (start 234.95 101.6) (end 247.65 101.6) (layer F.SilkS) (width 0.12))
-  (gr_line (start 234.95 109.22) (end 247.65 109.22) (layer F.SilkS) (width 0.12))
-  (gr_line (start 234.95 116.84) (end 247.65 116.84) (layer F.SilkS) (width 0.12))
-  (gr_line (start 234.95 124.46) (end 247.65 124.46) (layer F.SilkS) (width 0.12))
-  (gr_line (start 234.95 132.08) (end 247.65 132.08) (layer F.SilkS) (width 0.12))
-  (gr_text AA (at 246.38 120.65 90) (layer F.SilkS)
+  (gr_line (start 234.95 72.39) (end 247.65 72.39) (layer F.SilkS) (width 0.12))
+  (gr_line (start 244.602 142.24) (end 244.602 42.291) (layer F.SilkS) (width 0.12))
+  (gr_line (start 234.95 80.01) (end 247.65 80.01) (layer F.SilkS) (width 0.12))
+  (gr_line (start 234.95 87.63) (end 247.65 87.63) (layer F.SilkS) (width 0.12))
+  (gr_line (start 234.95 95.25) (end 247.65 95.25) (layer F.SilkS) (width 0.12))
+  (gr_line (start 234.95 102.87) (end 247.65 102.87) (layer F.SilkS) (width 0.12))
+  (gr_line (start 234.95 110.49) (end 247.65 110.49) (layer F.SilkS) (width 0.12))
+  (gr_line (start 234.95 118.11) (end 247.65 118.11) (layer F.SilkS) (width 0.12))
+  (gr_line (start 234.95 125.73) (end 247.65 125.73) (layer F.SilkS) (width 0.12))
+  (gr_line (start 234.95 133.35) (end 247.65 133.35) (layer F.SilkS) (width 0.12))
+  (gr_text AA (at 246.38 121.92 90) (layer F.SilkS)
     (effects (font (size 1 1) (thickness 0.15)))
   )
@@
     (effects (font (size 1 1) (thickness 0.15)))
   )
-  (gr_text TX (at 246.38 90.17 90) (layer F.SilkS)
+  (gr_text TX (at 246.38 91.44 90) (layer F.SilkS)
     (effects (font (size 1 1) (thickness 0.15)))
   )
-  (gr_text "RX\n" (at 246.38 97.79 90) (layer F.SilkS)
+  (gr_text "RX\n" (at 246.38 99.06 90) (layer F.SilkS)
     (effects (font (size 1 1) (thickness 0.15)))
   )
-  (gr_text CD (at 246.38 113.03 90) (layer F.SilkS)
+  (gr_text CD (at 246.38 114.3 90) (layer F.SilkS)
     (effects (font (size 1 1) (thickness 0.15)))
   )
-  (gr_text "OH\n" (at 246.38 105.41 90) (layer F.SilkS)
+  (gr_text "OH\n" (at 246.38 106.68 90) (layer F.SilkS)
     (effects (font (size 1 1) (thickness 0.15)))
   )
-  (gr_text RI (at 246.38 128.27 90) (layer F.SilkS)
+  (gr_text RI (at 246.38 129.54 90) (layer F.SilkS)
     (effects (font (size 1 1) (thickness 0.15)))
   )
-  (gr_text DTR (at 246.38 82.55 90) (layer F.SilkS)
+  (gr_text DTR (at 246.38 83.82 90) (layer F.SilkS)
     (effects (font (size 1 1) (thickness 0.15)))
   )

Commit message: updates
Parts:
- removed the REF** at (241.3, 123.2)
- removed the REF** at (241.3, 130.8)
- added REF**: Pin_Header_Straight_2x10_Pitch2.54mm, Pin_Headers:Pin_Header_Straight_2x10_Pitch2.54mm, F.Cu at (189.2, 128.3)
- added REF**: LED_D3.0mm, LEDs:LED_D3.0mm, F.Cu at (240.0, 105.4)
- added REF**: LED_D3.0mm, LEDs:LED_D3.0mm, F.Cu at (240.0, 113.0)
- added REF**: Pin_Header_Straight_1x08_Pitch2.54mm, Pin_Headers:Pin_Header_Straight_1x08_Pitch2.54mm, F.Cu at (138.4, 148.6)
- added REF**: Pin_Header_Straight_1x08_Pitch2.54mm, Pin_Headers:Pin_Header_Straight_1x08_Pitch2.54mm, F.Cu at (77.5, 148.6)
- added REF**: Pin_Header_Straight_2x10_Pitch2.54mm, Pin_Headers:Pin_Header_Straight_2x10_Pitch2.54mm, F.Cu at (128.3, 128.3)
- moved REF** 34.9 mm to (182.9, 54.6)
- moved REF** 34.9 mm to (202.5, 54.2)
- moved REF** 34.7 mm to (146.1, 100.3), turned to 270 degrees
- moved REF** 25.2 mm to (154.9, 45.7)
- moved REF** 22.9 mm to (168.9, 114.3)
- moved REF** 22.3 mm to (154.9, 80.0)
- moved REF** 19.4 mm to (104.7, 66.0)
- moved REF** 17.8 mm to (207.0, 31.5)
- moved DB_9F 17.8 mm to (78.0, 100.1)
- moved REF** 17.8 mm to (215.9, 35.6)
- moved REF** 17.8 mm to (238.8, 35.6)
- moved REF** 17.8 mm to (240.0, 67.3)
- moved REF** 17.8 mm to (240.0, 82.5)
- moved REF** 17.8 mm to (240.0, 90.2)
- moved REF** 17.8 mm to (187.6, 38.2)
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Other:
- board size 172.7 x 100 mm -> 172.7 x 130.5 mm
- board text added: "AUTO"
- board text added: "DT/CE"
- board text added: "HI-Z"
- board text added: "SHUTDOWN"
- board text removed: "DCE"
- board text removed: "DTE"

Commit message: updates
Parts:
- added REF**: MountingHole_2.5mm_Pad_Via, Mounting_Holes:MountingHole_2.5mm_Pad_Via, F.Cu at (240.0, 150.5)
Other:
- outline, holes or cut-outs redrawn
- board text added: "hegars.com"
- board text added: "pcb@hegars.com"
- board text added: "uCctl"
- board text removed: "AUTO"
