File: 300BaudModem.sch (KiCad schematic (older format))
At the start: 1 part

Commit message: working on it still
Parts:
- added BZ?: Buzzer, symbol Device:Buzzer
- added C? (x2): 3u3, symbol Device:C_Polarized
- added C? (x5): 100n, symbol Device:C
- added C?: C, symbol Device:C
- added C? (x2): 100u, symbol Device:C_Polarized
- added D?: RX, symbol Device:LED
- added D?: TX, symbol Device:LED
- added D?: CD, symbol Device:LED
- added D?: OH, symbol Device:LED
- added D?: RI, symbol Device:LED
- added D?: PWR, symbol Device:LED
- added Q?: Q_PMOS_SDG, symbol Device:Q_PMOS_SDG
- added R? (x2): 10K, symbol Device:R
- added R? (x2): R, symbol Device:R
- added R? (x7): 1K, symbol Device:R
- added R?: 100, symbol Device:R
- added R? (x2): 220, symbol Device:R
- added RV?: 100k, symbol Device:R_Potentiometer
- added SW?: SW_Push, symbol Switch:SW_Push
- added U?: 74LS14, symbol 74xx:74LS14
- added Y?: 16Mhz, symbol Device:Crystal
Connections:
- net labels added: +5V, Baseband-IN, Baseband-OUT, GND, Mega-AREF, Mega-PB0, Mega-PB1, Mega-PB2, Mega-PB3, Mega-PB4, Mega-PB5, Mega-PC0, Mega-PD0, Mega-PD1, Mega-PD2, Mega-PD3, Mega-PD4, Mega-PD5, Mega-PD6, Mega-PD7, Mega-RST, Mega-XTAL1, Mega-XTAL2, RST_REQ, TTL-CTS, TTL-DCD, TTL-DSR, TTL-DTR, TTL-RI, TTL-RTS, TTL-RX, TTL-TX
- wire segments 0 -> 34
Other:
- note added: "BUS to TTL"
- note added: "Baseband Inbound"
- note added: "Baseband Outbound"
- note added: "Baseband Outbound Monitor (ATM1)"
- note added: "CLOCK"
- note added: "ICSP"
- note added: "Indications"
- note added: "Reset w/Watchdog access"
- note added: "uController"

Commit message: updates
Parts:
- added C?: 100n, symbol Device:C
- added J?: Conn_02x03_Odd_Even, symbol Connector_Generic:Conn_02x03_Odd_Even
- U?: symbol MCU_Microchip_ATmega:ATmega328-P -> MCU_Microchip_ATmega:ATmega328P-A
Other:
- note added: "Baseband Monitor via AT (ATM1)"
- note removed: "Baseband Outbound Monitor (ATM1)"
Changed lines of the file:
@@
 $EndDescr
 $Comp
-L MCU_Microchip_ATmega:ATmega328-P U?
+L MCU_Microchip_ATmega:ATmega328P-A U?
 U 1 1 60DF35F3
 P 6050 3250
@@
 Connection ~ 2950 4800
 Wire Wire Line
-	2050 4300 2050 4350
-Wire Wire Line
-	2050 4350 2400 4350
-Wire Wire Line
-	2400 4350 2400 4800
-Wire Wire Line
 	2050 4000 3500 4000
 $Comp
@@
 Wire Notes Line
 	1000 3500 4500 3500
-Connection ~ 2050 4300
 $Comp
 L power:GND #PWR?
@@
 Text GLabel 6650 2950 2    50   Input ~ 0
 Mega-PC0
-Text GLabel 5450 2050 0    50   Input ~ 0
+Text GLabel 5050 2050 0    50   Input ~ 0
 Mega-AREF
 Text GLabel 6650 2350 2    50   Input ~ 0
@@
 Text Notes 1100 1150 0    50   ~ 0
 Indications
-Text Notes 1100 3650 0    50   ~ 0
+Text Notes 1050 3650 0    50   ~ 0
 Baseband Inbound
-Text Notes 3050 1150 0    50   ~ 0
+Text Notes 3100 1150 0    50   ~ 0
 BUS to TTL
-Text Notes 1100 5700 0    50   ~ 0
+Text Notes 1050 5650 0    50   ~ 0
 Baseband Outbound
-Text Notes 1150 6900 0    50   ~ 0
-Baseband Outbound Monitor (ATM1)
+Text Notes 1050 6900 0    50   ~ 0
+Baseband Monitor via AT (ATM1)
 $Comp
 L Switch:SW_Push SW?
@@
 Text Notes 7950 2650 0    50   ~ 0
 CLOCK
-Text Notes 9650 2650 0    50   ~ 0
+Text Notes 7950 3650 0    50   ~ 0
 ICSP
-Wire Notes Line
-	9500 3500 9500 2500
 Wire Notes Line
 	10750 1000 10750 3500
@@
 Wire Wire Line
 	8450 2900 8800 2900
+$Comp
+L Connector_Generic:Conn_02x03_Odd_Even J?
+U 1 1 60EEF453
+P 8600 4100
+F 0 "J?" H 8650 4417 50  0000 C CNN
+F 1 "Conn_02x03_Odd_Even" H 8650 4326 50  0000 C CNN
+F 2 "" H 8600 4100 50  0001 C CNN
+F 3 "~" H 8600 4100 50  0001 C CNN
+	1    8600 4100
+	1    0    0    -1
+$EndComp
+$Comp
+L power:GND #PWR?
+U 1 1 60EF013C
+P 8900 4200
+F 0 "#PWR?" H 8900 3950 50  0001 C CNN
+F 1 "GND" V 8905 4072 50  0000 R CNN
+F 2 "" H 8900 4200 50  0001 C CNN
+F 3 "" H 8900 4200 50  0001 C CNN
+	1    8900 4200
+	0    -1   -1   0
+$EndComp
+$Comp
+L power:+5V #PWR?
+U 1 1 60EF0858
+P 8900 4000
+F 0 "#PWR?" H 8900 3850 50  0001 C CNN
+F 1 "+5V" V 8915 4128 50  0000 L CNN
+F 2 "" H 8900 4000 50  0001 C CNN
+F 3 "" H 8900 4000 50  0001 C CNN
+	1    8900 4000
+	0    1    1    0
+$EndComp
+Text GLabel 8900 4100 2    50   Input ~ 0
+Mega-PB3
+Text GLabel 8400 4200 0    50   Input ~ 0
+Mega-RST
+Text GLabel 8400 4100 0    50   Input ~ 0
+Mega-PB5
+Text GLabel 8400 4000 0    50   Input ~ 0
+Mega-PB4
+Wire Notes Line
+	9500 4500 7850 4500
+Wire Notes Line
+	9500 2500 9500 4500
+Wire Wire Line
+	2050 4300 2400 4300
+Connection ~ 2050 4300
+Wire Wire Line
+	2400 4300 2400 4800
+$Comp
+L Device:C C?
+U 1 1 60EF7F24
+P 5300 2050
+F 0 "C?" V 5048 2050 50  0000 C CNN
+F 1 "100n" V 5139 2050 50  0000 C CNN
+F 2 "" H 5338 1900 50  0001 C CNN
+F 3 "~" H 5300 2050 50  0001 C CNN
+	1    5300 2050
+	0    1    1    0
+$EndComp
+$Comp
+L power:GND #PWR?
+U 1 1 60EF8CF4
+P 5150 2050
+F 0 "#PWR?" H 5150 1800 50  0001 C CNN
+F 1 "GND" H 5155 1877 50  0000 C CNN
+F 2 "" H 5150 2050 50  0001 C CNN
+F 3 "" H 5150 2050 50  0001 C CNN
+	1    5150 2050
+	1    0    0    -1
+$EndComp
+Wire Wire Line
+	5050 2050 5150 2050
+Connection ~ 5150 2050
 $EndSCHEMATC

Commit message: updates
Parts:
- removed C?: 100u, symbol Device:C_Polarized
- removed Q?: Q_PMOS_SDG, symbol Device:Q_PMOS_SDG
- removed R?: 10K, symbol Device:R
- removed U?: 74LS14, symbol 74xx:74LS14
- added C? (x2): 1uf, symbol Device:C
- added C?: 100u, symbol Device:C_Polarized
- added C? (x2): 4.7uF, symbol Device:C_Polarized
- added Q?: Q_PMOS_SDG, symbol Device:Q_PMOS_SDG
- added R?: 220, symbol Device:R
- added R?: 10K, symbol Device:R
- added SW?: SW_Push, symbol Switch:SW_Push
- added U?: 74LS14, symbol 74xx:74LS14
- added U?: LM7805_TO220, Package_TO_SOT_THT:TO-220-3_Vertical, symbol Regulator_Linear:LM7805_TO220
- C?: value 100u -> 4.7uF
- R?: value 220 -> 1K
Connections:
- net +5V: now also R?.1, U?.18 (AVCC), C?.1, C?.1, C?.1, C?.1, U?.3 (VO)
- net GND: now also SW?.2, C?.2, C?.2, C?.2, C?.2, U?.2 (GND)
- net Mega-RST: now also SW?.1, R?.2
- net RST_REQ: now also U?.1
- new net: Q?.2 (D), R?.1, SW?.1
- new net: C?.2, Q?.1 (S), R?.2, SW?.2
- new net: Q?.3 (G), R?.1, U?.2
- new net +12V: C?.1, U?.1 (VI)
Other:
- note added: "Power Regulator (CHECK)"
- note added: "Reset"
- note added: "uC to TTL"
- note removed: "BUS to TTL"
- note removed: "Reset w/Watchdog access"
- moved on the sheet: C?, D?, R?, SW?

Commit message: updates
Parts:
- added J?: Conn_01x08_Male, symbol Connector:Conn_01x08_Male
- added J?: Conn_02x10_Odd_Even, symbol Connector_Generic:Conn_02x10_Odd_Even
- added J?: RJ45, symbol Connector:RJ45
- added J?: AudioPlug4, symbol Connector:AudioPlug4
Connections:
- net +5V: now also J?.1 (Pin_1), J?.2 (Pin_2)
- net Baseband-IN: now also J?.10 (Pin_10), J?.R1
- net Baseband-OUT: now also J?.12 (Pin_12), J?.T
- net GND: now also J?.19 (Pin_19), J?.20 (Pin_20), J?.S
- net Mega-PD0: now also J?.3 (Pin_3)
- net Mega-PD1: now also J?.5 (Pin_5)
- net Mega-PD2: now also J?.7 (Pin_7)
- net Mega-PD4: now also J?.9 (Pin_9)
- net Mega-PD5: now also J?.11 (Pin_11)
- net Mega-PD6: now also J?.13 (Pin_13)
- net Mega-PD7: now also J?.15 (Pin_15)
- net TTL-DCD: now also J?.17 (Pin_17)
- new net E&M-E: J?.2, J?.2 (Pin_2)
- new net E&M-M: J?.7, J?.7 (Pin_7)
- new net E&M-R: J?.4, J?.4 (Pin_4)
- new net E&M-R1: J?.3, J?.3 (Pin_3)
- new net E&M-SB: J?.1, J?.1 (Pin_1)
- new net E&M-SG: J?.8, J?.8 (Pin_8)
- new net E&M-T: J?.5, J?.5 (Pin_5)
- new net E&M-T1: J?.6, J?.6 (Pin_6)
- new net Signaling-OFFHOOK: J?.16 (Pin_16), J?.R2
- new net Signaling-RING: J?.6 (Pin_6)
Other:
- note added: "Audio Jack"
- note added: "Baseband Monitor (via AT Command "M1")"
- note added: "Reset (Pullup)"
- note added: "Telephony Module Interface E&M Type"
- note added: "Test Reset Circuit"
- note removed: "Baseband Monitor via AT (ATM1)"
- note removed: "Reset"
- moved on the sheet: BZ?, C?, D?, J?, Q?, R?, RV?, SW?, U?, U?A, Y?

Commit message: updates
Parts:
- added F? (x2): Polyfuse, symbol Device:Polyfuse
- added J?: Jack-DC, symbol Connector:Jack-DC
- J?: symbol Connector:Conn_01x08_Male -> Connector_Generic:Conn_01x08
Connections:
- net E&M-E: now also J?.7, J?.7 (Pin_7); no longer J?.2, J?.2 (Pin_2)
- net E&M-M: now also J?.2, J?.2 (Pin_2); no longer J?.7, J?.7 (Pin_7)
- net GND: now also J?.2
- net Mega-PD0: now also J?.9 (Pin_9); no longer J?.3 (Pin_3)
- net Mega-PD1: now also J?.11 (Pin_11); no longer J?.5 (Pin_5)
- net Mega-PD2: now also J?.5 (Pin_5); no longer J?.7 (Pin_7)
- net Mega-PD4: now also J?.3 (Pin_3); no longer J?.9 (Pin_9)
- net Mega-PD5: now also J?.17 (Pin_17); no longer J?.11 (Pin_11)
- net Mega-PD6: now also J?.7 (Pin_7); no longer J?.13 (Pin_13)
- net Mega-PD7: now also J?.13 (Pin_13); no longer J?.15 (Pin_15)
- net TTL-DCD: now also J?.15 (Pin_15); no longer J?.17 (Pin_17)
- net +12V: no longer names the net of C?.1, U?.1 (VI)
- net +12V: now also F?.2
- new net: F?.1, J?.1
Other:
- note added: "Backplane"
- note added: "E&M Type Output interface"
- note added: "Module Interface"
- note added: "TEST Reset Circuit"
- note added: "TTL to RS232"
- note removed: "Telephony Module Interface E&M Type"
- note removed: "Test Reset Circuit"
- moved on the sheet: C?, D?, J?, R?, U?, Y?

Commit message: updates
Connections:
- net Mega-RST: now also J?.4 (Pin_4)
- net Signaling-OFFHOOK: now also J?.14 (Pin_14); no longer J?.16 (Pin_16)
- net I2C-SDA: now reaches J?.18 (Pin_18)
- net Signaling-RINGING: now reaches J?.8 (Pin_8)
- net Mega-PD0 renamed TTL-RX
- net Mega-PD1 renamed TTL-TX
- net Mega-PD2 renamed TTL-RI
- net Mega-PD4 renamed TTL-DTR
- net Mega-PD5 renamed TTL-DSR
- net Mega-PD6 renamed TTL-RTS
- net Mega-PD7 renamed TTL-CTS
- net Signaling-RING: no longer names the net of J?.6 (Pin_6)
- new net I2C-SDL: J?.16 (Pin_16)
Other:
- note added: "Baseband Input (Needs Work)"
- note added: "Baseband Monitor (via AT Command "M0/1")"
- note added: "Baseband Output"
- note removed: "Baseband Inbound"
- note removed: "Baseband Monitor (via AT Command "M1")"
- note removed: "Baseband Outbound"
- note removed: "uC to TTL"
- moved on the sheet: J?
Changed lines of the file:
@@
 Wire Notes Line
 	550  550  550  7050
-Text GLabel 9650 3750 2    50   Input ~ 0
-Mega-PD6
-Text GLabel 9650 3750 0    50   Input ~ 0
+Text GLabel 6400 4350 2    50   Input ~ 0
 TTL-RTS
-Text GLabel 9650 3850 0    50   Input ~ 0
+Text GLabel 6400 4450 2    50   Input ~ 0
 TTL-CTS
-Text GLabel 9650 3550 0    50   Input ~ 0
+Text GLabel 6400 4150 2    50   Input ~ 0
 TTL-DTR
-Text GLabel 9650 3650 0    50   Input ~ 0
+Text GLabel 6400 4250 2    50   Input ~ 0
 TTL-DSR
-Text GLabel 9650 3350 0    50   Input ~ 0
+Text GLabel 6400 3850 2    50   Input ~ 0
 TTL-TX
-Text GLabel 9650 3250 0    50   Input ~ 0
+Text GLabel 6400 3750 2    50   Input ~ 0
 TTL-RX
-Text GLabel 9650 3950 0    50   Input ~ 0
+Text GLabel 6400 4550 2    50   Input ~ 0
 TTL-DCD
-Text GLabel 9650 3450 0    50   Input ~ 0
+Text GLabel 6400 3950 2    50   Input ~ 0
 TTL-RI
-Text GLabel 9650 3850 2    50   Input ~ 0
-Mega-PD7
-Text GLabel 9650 3550 2    50   Input ~ 0
-Mega-PD4
-Text GLabel 9650 3650 2    50   Input ~ 0
-Mega-PD5
-Text GLabel 9650 3450 2    50   Input ~ 0
-Mega-PD2
-Text GLabel 9650 3350 2    50   Input ~ 0
-Mega-PD1
-Text GLabel 9650 3250 2    50   Input ~ 0
-Mega-PD0
-Text GLabel 6400 4350 2    50   Input ~ 0
-Mega-PD6
-Text GLabel 6400 4450 2    50   Input ~ 0
-Mega-PD7
-Text GLabel 6400 4150 2    50   Input ~ 0
-Mega-PD4
-Text GLabel 6400 4250 2    50   Input ~ 0
-Mega-PD5
-Text GLabel 6400 3950 2    50   Input ~ 0
-Mega-PD2
-Text GLabel 6400 3850 2    50   Input ~ 0
-Mega-PD1
-Text GLabel 6400 3750 2    50   Input ~ 0
-Mega-PD0
 Text GLabel 6400 2050 2    50   Input ~ 0
 Mega-PB0
@@
 Text GLabel 6400 2350 2    50   Input ~ 0
 Mega-PB3
-Text GLabel 6400 4050 2    50   Input ~ 0
-Mega-PD3
 $Comp
 L Device:Crystal Y?
@@
 Indications
 Text Notes 600  3200 0    50   ~ 0
-Baseband Inbound
-Text Notes 9100 3150 0    50   ~ 0
-uC to TTL
+Baseband Input (Needs Work)
 Text Notes 600  5200 0    50   ~ 0
-Baseband Outbound
+Baseband Output
 Text Notes 600  6450 0    50   ~ 0
-Baseband Monitor (via AT Command "M1")
+Baseband Monitor (via AT Command "M0/1")
 $Comp
 L Switch:SW_Push SW?
@@
 L Connector_Generic:Conn_02x03_Odd_Even J?
 U 1 1 60EEF453
-P 8200 3650
-F 0 "J?" H 8250 3967 50  0000 C CNN
-F 1 "Conn_02x03_Odd_Even" H 8250 3876 50  0000 C CNN
-F 2 "" H 8200 3650 50  0001 C CNN
-F 3 "~" H 8200 3650 50  0001 C CNN
-	1    8200 3650
+P 8850 3650
+F 0 "J?" H 8900 3967 50  0000 C CNN
+F 1 "Conn_02x03_Odd_Even" H 8900 3876 50  0000 C CNN
+F 2 "" H 8850 3650 50  0001 C CNN
+F 3 "~" H 8850 3650 50  0001 C CNN
+	1    8850 3650
 	1    0    0    -1
 $EndComp
@@
 L power:GND #PWR?
 U 1 1 60EF013C
-P 8500 3750
-F 0 "#PWR?" H 8500 3500 50  0001 C CNN
-F 1 "GND" V 8505 3622 50  0000 R CNN
-F 2 "" H 8500 3750 50  0001 C CNN
-F 3 "" H 8500 3750 50  0001 C CNN
-	1    8500 3750
+P 9150 3750
+F 0 "#PWR?" H 9150 3500 50  0001 C CNN
+F 1 "GND" V 9155 3622 50  0000 R CNN
+F 2 "" H 9150 3750 50  0001 C CNN
+F 3 "" H 9150 3750 50  0001 C CNN
+	1    9150 3750
 	0    -1   -1   0
 $EndComp
@@
 L power:+5V #PWR?
 U 1 1 60EF0858
-P 8500 3550
-F 0 "#PWR?" H 8500 3400 50  0001 C CNN
-F 1 "+5V" V 8515 3678 50  0000 L CNN
-F 2 "" H 8500 3550 50  0001 C CNN
-F 3 "" H 8500 3550 50  0001 C CNN
-	1    8500 3550
-	0    1    1    0
-$EndComp
-Text GLabel 8500 3650 2    50   Input ~ 0
+P 9150 3550
+F 0 "#PWR?" H 9150 3400 50  0001 C CNN
+F 1 "+5V" V 9165 3678 50  0000 L CNN
+F 2 "" H 9150 3550 50  0001 C CNN
+F 3 "" H 9150 3550 50  0001 C CNN
+	1    9150 3550
+	0    1    1    0
+$EndComp
+Text GLabel 9150 3650 2    50   Input ~ 0
 Mega-PB3
-Text GLabel 8000 3750 0    50   Input ~ 0
+Text GLabel 8650 3750 0    50   Input ~ 0
 Mega-RST
-Text GLabel 8000 3650 0    50   Input ~ 0
+Text GLabel 8650 3650 0    50   Input ~ 0
 Mega-PB5
-Text GLabel 8000 3550 0    50   Input ~ 0
+Text GLabel 8650 3550 0    50   Input ~ 0
 Mega-PB4
 Wire Wire Line
@@
 L power:GND #PWR?
 U 1 1 60F3E40B
-P 9400 1250
-F 0 "#PWR?" H 9400 1000 50  0001 C CNN
-F 1 "GND" V 9405 1122 50  0000 R CNN
-F 2 "" H 9400 1250 50  0001 C CNN
-F 3 "" H 9400 1250 50  0001 C CNN
-	1    9400 1250
-	0    -1   -1   0
+P 9650 1550
+F 0 "#PWR?" H 9650 1300 50  0001 C CNN
+F 1 "GND" V 9655 1422 50  0000 R CNN
+F 2 "" H 9650 1550 50  0001 C CNN
+F 3 "" H 9650 1550 50  0001 C CNN
+	1    9650 1550
+	1    0    0    -1
 $EndComp
 Wire Wire Line
@@
 L Connector:AudioPlug4 J?
 U 1 1 60F81E30
-P 8100 4600
-F 0 "J?" H 8157 4925 50  0000 C CNN
-F 1 "AudioPlug4" H 8157 4834 50  0000 C CNN
-F 2 "" H 8450 4500 50  0001 C CNN
-F 3 "~" H 8450 4500 50  0001 C CNN
-	1    8100 4600
+P 8500 4550
+F 0 "J?" H 8557 4875 50  0000 C CNN
+F 1 "AudioPlug4" H 8557 4784 50  0000 C CNN
+F 2 "" H 8850 4450 50  0001 C CNN
+F 3 "~" H 8850 4450 50  0001 C CNN
+	1    8500 4550
 	1    0    0    -1
 $EndComp
@@
 L power:GND #PWR?
 U 1 1 60F83B3F
-P 8700 4500
-F 0 "#PWR?" H 8700 4250 50  0001 C CNN
-F 1 "GND" V 8705 4372 50  0000 R CNN
-F 2 "" H 8700 4500 50  0001 C CNN
-F 3 "" H 8700 4500 50  0001 C CNN
-	1    8700 4500
+P 9100 4450
+F 0 "#PWR?" H 9100 4200 50  0001 C CNN
+F 1 "GND" V 9105 4322 50  0000 R CNN
+F 2 "" H 9100 4450 50  0001 C CNN
+F 3 "" H 9100 4450 50  0001 C CNN
+	1    9100 4450
 	0    -1   -1   0
 $EndComp
-Text GLabel 8700 4800 2    50   Input ~ 0
+Text GLabel 9100 4750 2    50   Input ~ 0
 Baseband-OUT
-Text GLabel 8700 4700 2    50   Output ~ 0
+Text GLabel 9100 4650 2    50   Output ~ 0
 Baseband-IN
 Text Notes 7500 4250 0    50   ~ 0
 Audio Jack
-Text GLabel 8700 4600 2    50   Input ~ 0
+Text GLabel 9100 4550 2    50   Input ~ 0
 Signaling-OFFHOOK
 Wire Wire Line
@@
 Wire Notes Line
 	7400 3050 10300 3050
-Wire Notes Line
-	9050 4050 9050 3050
 Wire Notes Line
 	550  5050 10300 5050
@@
 Text GLabel 5650 5900 2    50   Output ~ 0
 Baseband-OUT
-Text GLabel 5650 6100 2    50   Input ~ 0
+Text GLabel 5650 6000 2    50   Input ~ 0
 Signaling-OFFHOOK
 Text GLabel 5150 5700 0    50   Input ~ 0
@@
 Wire Notes Line
 	550  7050 4050 7050
-Text GLabel 5650 5600 2    50   Output ~ 0
-Signaling-RING
+Text GLabel 5650 5700 2    50   Output ~ 0
+Signaling-RINGING
 Wire Notes Line
 	10300 550  10300 6450
@@
 	2700 1650 2700 2250
 Connection ~ 2700 2250
+Wire Wire Line
+	9650 1550 9650 1250
+Wire Wire Line
+	9400 1250 9650 1250
+Text GLabel 5650 5500 2    50   Output ~ 0
+Mega-RST
+Text GLabel 5650 6100 2    50   Input ~ 0
+I2C-SDL
+Text GLabel 5650 6200 2    50   Input ~ 0
+I2C-SDA
+Text GLabel 6400 4800 2    50   Input ~ 0
+I2C-SDL
+Text GLabel 6400 4900 2    50   Input ~ 0
+I2C-SDA
+Text GLabel 6400 4050 2    50   Input ~ 0
+Mega-PD3
 $EndSCHEMATC
