File: 300BaudModem.sch (KiCad schematic (older format))
At the start: 0 parts

Commit message: more updates
Changed lines of the file:
@@
 $EndDescr
 $Sheet
-S 2500 2500 1000 1000
+S 9800 2550 1000 1000
 U 60E5C27B
 F0 "PCMBus" 50
@@
 $EndSheet
 $Sheet
-S 2500 1000 1000 1000
+S 9800 1050 1000 1000
 U 60E5CADB
 F0 "ECBus" 50

Commit message: updates
Changed lines of the file:
@@
 $Descr A4 11693 8268
 encoding utf-8
-Sheet 1 10
+Sheet 1 11
 Title "300 Baud Audio FSK Modem "
 Date "2021-07-08"
@@
 $EndDescr
 $Sheet
-S 9800 2550 1000 1000
+S 9500 2500 1000 1000
 U 60E5C27B
 F0 "PCMBus" 50
@@
 $EndSheet
 $Sheet
-S 9800 1050 1000 1000
+S 9500 1000 1000 1000
 U 60E5CADB
 F0 "ECBus" 50
@@
 F1 "RS232.sch" 50
 $EndSheet
+$Sheet
+S 9500 4000 1000 1050
+U 60F27560
+F0 "Serial2WiFI" 50
+F1 "Ser2WIFI.sch" 50
+$EndSheet
 $EndSCHEMATC

Commit message: general updates
Changed lines of the file:
@@
 $Descr A4 11693 8268
 encoding utf-8
-Sheet 1 11
+Sheet 1 12
 Title "300 Baud Audio FSK Modem "
 Date "2021-07-08"
@@
 F1 "Ser2WIFI.sch" 50
 $EndSheet
+$Sheet
+S 4500 5650 1000 900
+U 60FC6F01
+F0 "hybrid" 50
+F1 "hybrid.sch" 50
+$EndSheet
 $EndSCHEMATC
