File: _autosave-Indications.sch (KiCad schematic (older format))
At the start: 30 parts

Commit message: general updates
Connections:
- net +5V: now also R?.1; no longer D?.1 (K)
- net GND: now also D?.1 (K); no longer R?.1
Other:
- moved on the sheet: D?, R?
Changed lines of the file:
@@
 L Device:R R?
 U 1 1 60EFCDA3
-P 8700 2950
+P 8400 2950
 AR Path="/60EFCDA3" Ref="R?"  Part="1"
 AR Path="/60EBA1DA/60EFCDA3" Ref="R?"  Part="1"
-F 0 "R?" V 8493 2950 50  0000 C CNN
-F 1 "1K" V 8584 2950 50  0000 C CNN
-F 2 "" V 8630 2950 50  0001 C CNN
-F 3 "~" H 8700 2950 50  0001 C CNN
-	1    8700 2950
-	0    1    1    0
+F 0 "R?" V 8193 2950 50  0000 C CNN
+F 1 "1K" V 8284 2950 50  0000 C CNN
+F 2 "" V 8330 2950 50  0001 C CNN
+F 3 "~" H 8400 2950 50  0001 C CNN
+	1    8400 2950
+	0    -1   -1   0
 $EndComp
 $Comp
 L Device:LED D?
 U 1 1 60EFCDAD
-P 8400 2950
+P 8700 2950
 AR Path="/60EFCDAD" Ref="D?"  Part="1"
 AR Path="/60EBA1DA/60EFCDAD" Ref="D?"  Part="1"
-F 0 "D?" H 8393 3167 50  0000 C CNN
-F 1 "PWR" H 8393 3076 50  0000 C CNN
-F 2 "" H 8400 2950 50  0001 C CNN
-F 3 "~" H 8400 2950 50  0001 C CNN
-	1    8400 2950
-	1    0    0    -1
+F 0 "D?" H 8693 3167 50  0000 C CNN
+F 1 "PWR" H 8693 3076 50  0000 C CNN
+F 2 "" H 8700 2950 50  0001 C CNN
+F 3 "~" H 8700 2950 50  0001 C CNN
+	1    8700 2950
+	-1   0    0    1
 $EndComp
 $Comp
@@
 L power:+5V #PWR?
 U 1 1 60F16AD2
-P 8100 3500
+P 8100 2950
 AR Path="/60F16AD2" Ref="#PWR?"  Part="1"
 AR Path="/60EBA1DA/60F16AD2" Ref="#PWR?"  Part="1"
-F 0 "#PWR?" H 8100 3350 50  0001 C CNN
-F 1 "+5V" V 8115 3628 50  0000 L CNN
-F 2 "" H 8100 3500 50  0001 C CNN
-F 3 "" H 8100 3500 50  0001 C CNN
-	1    8100 3500
+F 0 "#PWR?" H 8100 2800 50  0001 C CNN
+F 1 "+5V" V 8115 3078 50  0000 L CNN
+F 2 "" H 8100 2950 50  0001 C CNN
+F 3 "" H 8100 2950 50  0001 C CNN
+	1    8100 2950
 	0    -1   -1   0
 $EndComp
@@
 Wire Wire Line
 	8350 3500 8100 3500
-Connection ~ 8100 3500
 $Comp
 L power:GND #PWR?
@@
 Wire Wire Line
 	9250 4850 9600 4850
+Connection ~ 8100 2950
 $EndSCHEMATC
