File: Indications.sch (KiCad schematic (older format))
At the start: 30 parts

Commit message: updates
Parts:
- added D?: DSR, symbol Device:LED
- added R?: 1K, symbol Device:R
- D?: value AUX1 -> AA
- D?: value AUX2 -> DTR
Connections:
- net +5V: now also R?.1; no longer D?.1 (K)
- net GND: now also D?.1 (K), D?.1 (K); no longer R?.1
- net at J?.9 (Pin_9): now also R?.1
- new net: D?.2 (A), R?.2
Other:
- moved on the sheet: D?, J?, R?
