File: Ser2WIFI.sch (KiCad schematic (older format))
At the start: 3 parts

Commit message: sch updates
Other:
- moved on the sheet: J?
Changed lines of the file:
@@
 L Connector:Conn_01x15_Female J?
 U 1 1 60F28A70
-P 4650 3800
-F 0 "J?" H 4542 2875 50  0000 C CNN
-F 1 "Conn_01x15_Female" H 4542 2966 50  0000 C CNN
-F 2 "" H 4650 3800 50  0001 C CNN
-F 3 "~" H 4650 3800 50  0001 C CNN
-	1    4650 3800
+P 4300 3750
+F 0 "J?" H 4192 2825 50  0000 C CNN
+F 1 "Conn_01x15_Female" H 4192 2916 50  0000 C CNN
+F 2 "" H 4300 3750 50  0001 C CNN
+F 3 "~" H 4300 3750 50  0001 C CNN
+	1    4300 3750
 	-1   0    0    1
 $EndComp
@@
 L Connector:Conn_01x15_Female J?
 U 1 1 60F2AD71
-P 7100 3800
-F 0 "J?" H 7128 3826 50  0000 L CNN
-F 1 "Conn_01x15_Female" H 7128 3735 50  0000 L CNN
-F 2 "" H 7100 3800 50  0001 C CNN
-F 3 "~" H 7100 3800 50  0001 C CNN
-	1    7100 3800
+P 7350 3750
+F 0 "J?" H 7378 3776 50  0000 L CNN
+F 1 "Conn_01x15_Female" H 7378 3685 50  0000 L CNN
+F 2 "" H 7350 3750 50  0001 C CNN
+F 3 "~" H 7350 3750 50  0001 C CNN
+	1    7350 3750
 	1    0    0    -1
 $EndComp
