File: hybrid.sch (KiCad schematic (older format))
At the start: 12 parts

Commit message: sch updates
Other:
- note added: "Network Buildout\n"
- moved on the sheet: C?, R?, T?
Changed lines of the file:
@@
 L Device:Transformer_1P_SS T?
 U 1 1 60FC799A
-P 4100 3200
-F 0 "T?" H 4100 3581 50  0000 C CNN
-F 1 "Transformer_1P_SS" H 4100 3490 50  0000 C CNN
-F 2 "" H 4100 3200 50  0001 C CNN
-F 3 "~" H 4100 3200 50  0001 C CNN
-	1    4100 3200
+P 4600 3450
+F 0 "T?" H 4600 3831 50  0000 C CNN
+F 1 "Transformer_1P_SS" H 4600 3740 50  0000 C CNN
+F 2 "" H 4600 3450 50  0001 C CNN
+F 3 "~" H 4600 3450 50  0001 C CNN
+	1    4600 3450
 	1    0    0    -1
 $EndComp
@@
 L Device:Transformer_1P_SS T?
 U 1 1 60FC83DF
-P 4100 4200
-F 0 "T?" H 4100 4581 50  0000 C CNN
-F 1 "Transformer_1P_SS" H 4100 4490 50  0000 C CNN
-F 2 "" H 4100 4200 50  0001 C CNN
-F 3 "~" H 4100 4200 50  0001 C CNN
-	1    4100 4200
+P 4600 4450
+F 0 "T?" H 4600 4831 50  0000 C CNN
+F 1 "Transformer_1P_SS" H 4600 4740 50  0000 C CNN
+F 2 "" H 4600 4450 50  0001 C CNN
+F 3 "~" H 4600 4450 50  0001 C CNN
+	1    4600 4450
 	1    0    0    -1
 $EndComp
@@
 L Device:Transformer_1P_SS T?
 U 1 1 60FC9250
-P 6400 4200
-F 0 "T?" H 6400 4581 50  0000 C CNN
-F 1 "Transformer_1P_SS" H 6400 4490 50  0000 C CNN
-F 2 "" H 6400 4200 50  0001 C CNN
-F 3 "~" H 6400 4200 50  0001 C CNN
-	1    6400 4200
+P 6900 4450
+F 0 "T?" H 6900 4831 50  0000 C CNN
+F 1 "Transformer_1P_SS" H 6900 4740 50  0000 C CNN
+F 2 "" H 6900 4450 50  0001 C CNN
+F 3 "~" H 6900 4450 50  0001 C CNN
+	1    6900 4450
 	-1   0    0    -1
 $EndComp
@@
 L Device:Transformer_1P_SS T?
 U 1 1 60FC9AF1
-P 6400 3200
-F 0 "T?" H 6400 3581 50  0000 C CNN
-F 1 "Transformer_1P_SS" H 6400 3490 50  0000 C CNN
-F 2 "" H 6400 3200 50  0001 C CNN
-F 3 "~" H 6400 3200 50  0001 C CNN
-	1    6400 3200
+P 6900 3450
+F 0 "T?" H 6900 3831 50  0000 C CNN
+F 1 "Transformer_1P_SS" H 6900 3740 50  0000 C CNN
+F 2 "" H 6900 3450 50  0001 C CNN
+F 3 "~" H 6900 3450 50  0001 C CNN
+	1    6900 3450
 	-1   0    0    -1
 $EndComp
 Wire Wire Line
-	4500 4000 6000 4000
-Wire Wire Line
-	6000 4400 5450 4400
-Wire Wire Line
-	5450 4400 5450 5500
-Wire Wire Line
-	4500 4400 5050 4400
-Wire Wire Line
-	5050 4400 5050 5500
-Wire Wire Line
-	4500 3400 5550 3400
-Wire Wire Line
-	5550 3400 5900 3000
-Wire Wire Line
-	5900 3000 6000 3000
-Wire Wire Line
-	3500 3400 3500 4000
-Wire Wire Line
-	3700 4400 3100 4400
-Wire Wire Line
-	3100 4400 3100 2500
-Wire Wire Line
-	3700 3000 3500 3000
-Wire Wire Line
-	3500 3000 3500 2900
-Wire Wire Line
-	6800 4400 7400 4400
-Wire Wire Line
-	6800 3000 7000 3000
-Wire Wire Line
-	7000 3000 7000 2700
+	5000 4250 6500 4250
+Wire Wire Line
+	6500 4650 5950 4650
+Wire Wire Line
+	5950 4650 5950 5750
+Wire Wire Line
+	5000 4650 5550 4650
+Wire Wire Line
+	5550 4650 5550 5750
+Wire Wire Line
+	5000 3650 6050 3650
+Wire Wire Line
+	6050 3650 6400 3250
+Wire Wire Line
+	6400 3250 6500 3250
+Wire Wire Line
+	4000 3650 4000 4250
+Wire Wire Line
+	4200 4650 3600 4650
+Wire Wire Line
+	3600 4650 3600 2750
+Wire Wire Line
+	4200 3250 4000 3250
+Wire Wire Line
+	4000 3250 4000 3150
+Wire Wire Line
+	7300 4650 7900 4650
+Wire Wire Line
+	7300 3250 7500 3250
+Wire Wire Line
+	7500 3250 7500 2950
 $Comp
 L Device:R R?
 U 1 1 60FD57B4
-P 7200 2700
-F 0 "R?" V 6993 2700 50  0000 C CNN
-F 1 "600" V 7084 2700 50  0000 C CNN
-F 2 "" V 7130 2700 50  0001 C CNN
-F 3 "~" H 7200 2700 50  0001 C CNN
-	1    7200 2700
+P 7700 2950
+F 0 "R?" V 7493 2950 50  0000 C CNN
+F 1 "600" V 7584 2950 50  0000 C CNN
+F 2 "" V 7630 2950 50  0001 C CNN
+F 3 "~" H 7700 2950 50  0001 C CNN
+	1    7700 2950
 	0    1    1    0
 $EndComp
@@
 L Device:R R?
 U 1 1 60FD6B73
-P 3500 2750
-F 0 "R?" H 3430 2704 50  0000 R CNN
-F 1 "600" H 3430 2795 50  0000 R CNN
-F 2 "" V 3430 2750 50  0001 C CNN
-F 3 "~" H 3500 2750 50  0001 C CNN
-	1    3500 2750
+P 4000 3000
+F 0 "R?" H 3930 2954 50  0000 R CNN
+F 1 "600" H 3930 3045 50  0000 R CNN
+F 2 "" V 3930 3000 50  0001 C CNN
+F 3 "~" H 4000 3000 50  0001 C CNN
+	1    4000 3000
 	-1   0    0    1
 $EndComp
 Wire Wire Line
-	3500 2600 3500 2500
+	4000 2850 4000 2750
 $Comp
 L Device:C C?
 U 1 1 60FD877E
-P 5100 2700
-F 0 "C?" H 4986 2654 50  0000 R CNN
-F 1 "120nF" H 4986 2745 50  0000 R CNN
-F 2 "" H 5138 2550 50  0001 C CNN
-F 3 "~" H 5100 2700 50  0001 C CNN
-	1    5100 2700
+P 5600 2950
+F 0 "C?" H 5486 2904 50  0000 R CNN
+F 1 "120nF" H 5486 2995 50  0000 R CNN
+F 2 "" H 5638 2800 50  0001 C CNN
+F 3 "~" H 5600 2950 50  0001 C CNN
+	1    5600 2950
 	0    -1   1    0
 $EndComp
 Wire Wire Line
-	5550 3000 5900 3400
+	6050 3250 6400 3650
 $Comp
 L Device:Transformer_1P_SS T?
 U 1 1 60FDF1F4
-P 3300 2100
-F 0 "T?" V 3346 2344 50  0000 L CNN
-F 1 "Transformer_1P_SS" V 3255 2344 50  0000 L CNN
-F 2 "" H 3300 2100 50  0001 C CNN
-F 3 "~" H 3300 2100 50  0001 C CNN
-	1    3300 2100
+P 3800 2350
+F 0 "T?" V 3846 2594 50  0000 L CNN
+F 1 "Transformer_1P_SS" V 3755 2594 50  0000 L CNN
+F 2 "" H 3800 2350 50  0001 C CNN
+F 3 "~" H 3800 2350 50  0001 C CNN
+	1    3800 2350
 	0    1    -1   0
 $EndComp
@@
 L Device:Transformer_1P_SS T?
 U 1 1 60FE15E2
-P 7200 2100
-F 0 "T?" V 7246 2344 50  0000 L CNN
-F 1 "Transformer_1P_SS" V 7155 2344 50  0000 L CNN
-F 2 "" H 7200 2100 50  0001 C CNN
-F 3 "~" H 7200 2100 50  0001 C CNN
-	1    7200 2100
+P 7700 2350
+F 0 "T?" V 7746 2594 50  0000 L CNN
+F 1 "Transformer_1P_SS" V 7655 2594 50  0000 L CNN
+F 2 "" H 7700 2350 50  0001 C CNN
+F 3 "~" H 7700 2350 50  0001 C CNN
+	1    7700 2350
 	0    1    -1   0
 $EndComp
@@
 L Device:Transformer_1P_SS T?
 U 1 1 60FECA17
-P 5250 5900
-F 0 "T?" V 5204 5612 50  0000 R CNN
-F 1 "Transformer_1P_SS" V 5295 5612 50  0000 R CNN
-F 2 "" H 5250 5900 50  0001 C CNN
-F 3 "~" H 5250 5900 50  0001 C CNN
-	1    5250 5900
+P 5750 6150
+F 0 "T?" V 5704 5862 50  0000 R CNN
+F 1 "Transformer_1P_SS" V 5795 5862 50  0000 R CNN
+F 2 "" H 5750 6150 50  0001 C CNN
+F 3 "~" H 5750 6150 50  0001 C CNN
+	1    5750 6150
 	0    -1   1    0
 $EndComp
 Wire Wire Line
-	4500 3000 4950 3000
+	5000 3250 5450 3250
 $Comp
 L Device:R R?
 U 1 1 60FF91B7
-P 5100 3000
-F 0 "R?" H 5030 2954 50  0000 R CNN
-F 1 "820" H 5030 3045 50  0000 R CNN
-F 2 "" V 5030 3000 50  0001 C CNN
-F 3 "~" H 5100 3000 50  0001 C CNN
-	1    5100 3000
+P 5600 3250
+F 0 "R?" H 5530 3204 50  0000 R CNN
+F 1 "820" H 5530 3295 50  0000 R CNN
+F 2 "" V 5530 3250 50  0001 C CNN
+F 3 "~" H 5600 3250 50  0001 C CNN
+	1    5600 3250
 	0    -1   -1   0
 $EndComp
@@
 L Device:R R?
 U 1 1 60FF98CB
-P 5400 3000
-F 0 "R?" H 5330 2954 50  0000 R CNN
-F 1 "220" H 5330 3045 50  0000 R CNN
-F 2 "" V 5330 3000 50  0001 C CNN
-F 3 "~" H 5400 3000 50  0001 C CNN
-	1    5400 3000
+P 5900 3250
+F 0 "R?" H 5830 3204 50  0000 R CNN
+F 1 "220" H 5830 3295 50  0000 R CNN
+F 2 "" V 5830 3250 50  0001 C CNN
+F 3 "~" H 5900 3250 50  0001 C CNN
+	1    5900 3250
 	0    -1   -1   0
 $EndComp
 Wire Wire Line
-	5250 2700 5250 3000
-Connection ~ 5250 3000
-Wire Wire Line
-	4950 3000 4950 2700
-Connection ~ 4950 3000
-Wire Wire Line
-	5900 3400 6000 3400
-Wire Wire Line
-	3500 4000 3700 4000
-Wire Wire Line
-	3500 3400 3700 3400
-Wire Wire Line
-	6800 3400 7000 3400
-Wire Wire Line
-	7000 3400 7000 4000
-Wire Wire Line
-	7000 4000 6800 4000
-Text Notes 3000 1600 0    50   ~ 0
+	5750 2950 5750 3250
+Connection ~ 5750 3250
+Wire Wire Line
+	5450 3250 5450 2950
+Connection ~ 5450 3250
+Wire Wire Line
+	6400 3650 6500 3650
+Wire Wire Line
+	4000 4250 4200 4250
+Wire Wire Line
+	4000 3650 4200 3650
+Wire Wire Line
+	7300 3650 7500 3650
+Wire Wire Line
+	7500 3650 7500 4250
+Wire Wire Line
+	7500 4250 7300 4250
+Text Notes 3500 1850 0    50   ~ 0
 4-Wire Transmit
-Text Notes 6900 1600 0    50   ~ 0
+Text Notes 7400 1850 0    50   ~ 0
 4-Wire Receive
-Text Notes 4800 6500 0    50   ~ 0
+Text Notes 5300 6750 0    50   ~ 0
 2-Wire Transmit/Receive
 Wire Wire Line
-	7400 2500 7400 2700
-Wire Wire Line
-	7050 2700 7000 2700
-Connection ~ 7000 2700
-Wire Wire Line
-	7000 2700 7000 2500
-Wire Wire Line
-	7350 2700 7400 2700
-Connection ~ 7400 2700
-Wire Wire Line
-	7400 2700 7400 4400
+	7900 2750 7900 2950
+Wire Wire Line
+	7550 2950 7500 2950
+Connection ~ 7500 2950
+Wire Wire Line
+	7500 2950 7500 2750
+Wire Wire Line
+	7850 2950 7900 2950
+Connection ~ 7900 2950
+Wire Wire Line
+	7900 2950 7900 4650
+Text Notes 5850 3100 0    50   ~ 0
+Network Buildout\n
 $EndSCHEMATC
