File: ECBus.sch (KiCad schematic (older format))
At the start: 0 parts

Commit message: updates
Parts:
- added J?: DIN41612_01x32_A, symbol Connector:DIN41612_01x32_A
Changed lines of the file:
@@
 Comment4 ""
 $EndDescr
+$Comp
+L Connector:DIN41612_01x32_A J?
+U 1 1 60E8EC77
+P 4850 3850
+F 0 "J?" H 4930 3842 50  0000 L CNN
+F 1 "DIN41612_01x32_A" H 4930 3751 50  0000 L CNN
+F 2 "" H 4850 3850 50  0001 C CNN
+F 3 "~" H 4850 3850 50  0001 C CNN
+	1    4850 3850
+	1    0    0    -1
+$EndComp
 $EndSCHEMATC

Commit message: updates
Parts:
- J?: symbol Connector:DIN41612_01x32_A -> Sebs:DIN41612_03x32_ABC
Connections:
- net +5V: now reaches J?.a1 (Pin_a1)
- net +5V: now also J?.b1 (Pin_b1), J?.c1 (Pin_c1)
- net +12V: now reaches J?.a13 (Pin_a13)
- net -12V: now reaches J?.a15 (Pin_a15)
- net +15V: now reaches J?.a19 (Pin_a19)
- net GND: now reaches J?.a32 (Pin_a32)
- net GND: now also J?.b32 (Pin_b32), J?.c32 (Pin_c32)
Changed lines of the file:
@@
 $EndDescr
 $Comp
-L Connector:DIN41612_01x32_A J?
+L Sebs:DIN41612_03x32_ABC J?
 U 1 1 60E8EC77
-P 4850 3850
-F 0 "J?" H 4930 3842 50  0000 L CNN
-F 1 "DIN41612_01x32_A" H 4930 3751 50  0000 L CNN
-F 2 "" H 4850 3850 50  0001 C CNN
-F 3 "~" H 4850 3850 50  0001 C CNN
-	1    4850 3850
+P 4550 3900
+F 0 "J?" H 4500 5550 50  0000 L CNN
+F 1 "DIN41612_01x32_A" H 4350 5650 50  0000 L CNN
+F 2 "" H 4550 3900 50  0001 C CNN
+F 3 "~" H 4550 3900 50  0001 C CNN
+	1    4550 3900
 	1    0    0    -1
 $EndComp
+$Comp
+L power:GND #PWR?
+U 1 1 61138E46
+P 3800 5450
+F 0 "#PWR?" H 3800 5200 50  0001 C CNN
+F 1 "GND" V 3805 5322 50  0000 R CNN
+F 2 "" H 3800 5450 50  0001 C CNN
+F 3 "" H 3800 5450 50  0001 C CNN
+	1    3800 5450
+	0    -1   -1   0
+$EndComp
+$Comp
+L power:+5V #PWR?
+U 1 1 611396B5
+P 3800 2350
+F 0 "#PWR?" H 3800 2200 50  0001 C CNN
+F 1 "+5V" V 3815 2478 50  0000 L CNN
+F 2 "" H 3800 2350 50  0001 C CNN
+F 3 "" H 3800 2350 50  0001 C CNN
+	1    3800 2350
+	0    1    1    0
+$EndComp
+$Comp
+L power:+5V #PWR?
+U 1 1 6113AD2B
+P 4800 2350
+F 0 "#PWR?" H 4800 2200 50  0001 C CNN
+F 1 "+5V" V 4815 2478 50  0000 L CNN
+F 2 "" H 4800 2350 50  0001 C CNN
+F 3 "" H 4800 2350 50  0001 C CNN
+	1    4800 2350
+	0    1    1    0
+$EndComp
+$Comp
+L power:GND #PWR?
+U 1 1 6113B70C
+P 5850 5450
+F 0 "#PWR?" H 5850 5200 50  0001 C CNN
+F 1 "GND" V 5855 5322 50  0000 R CNN
+F 2 "" H 5850 5450 50  0001 C CNN
+F 3 "" H 5850 5450 50  0001 C CNN
+	1    5850 5450
+	0    -1   -1   0
+$EndComp
+$Comp
+L power:GND #PWR?
+U 1 1 6113C54D
+P 4800 5450
+F 0 "#PWR?" H 4800 5200 50  0001 C CNN
+F 1 "GND" V 4805 5322 50  0000 R CNN
+F 2 "" H 4800 5450 50  0001 C CNN
+F 3 "" H 4800 5450 50  0001 C CNN
+	1    4800 5450
+	0    -1   -1   0
+$EndComp
+$Comp
+L power:+5V #PWR?
+U 1 1 6113D6D8
+P 5850 2350
+F 0 "#PWR?" H 5850 2200 50  0001 C CNN
+F 1 "+5V" V 5865 2478 50  0000 L CNN
+F 2 "" H 5850 2350 50  0001 C CNN
+F 3 "" H 5850 2350 50  0001 C CNN
+	1    5850 2350
+	0    1    1    0
+$EndComp
+$Comp
+L power:+12V #PWR?
+U 1 1 6113E23F
+P 3800 3550
+F 0 "#PWR?" H 3800 3400 50  0001 C CNN
+F 1 "+12V" V 3815 3678 50  0000 L CNN
+F 2 "" H 3800 3550 50  0001 C CNN
+F 3 "" H 3800 3550 50  0001 C CNN
+	1    3800 3550
+	0    1    1    0
+$EndComp
+$Comp
+L power:-12V #PWR?
+U 1 1 6113F43A
+P 3800 3750
+F 0 "#PWR?" H 3800 3850 50  0001 C CNN
+F 1 "-12V" V 3815 3878 50  0000 L CNN
+F 2 "" H 3800 3750 50  0001 C CNN
+F 3 "" H 3800 3750 50  0001 C CNN
+	1    3800 3750
+	0    1    1    0
+$EndComp
+$Comp
+L power:+15V #PWR?
+U 1 1 6114052C
+P 3800 4150
+F 0 "#PWR?" H 3800 4000 50  0001 C CNN
+F 1 "+15V" V 3815 4278 50  0000 L CNN
+F 2 "" H 3800 4150 50  0001 C CNN
+F 3 "" H 3800 4150 50  0001 C CNN
+	1    3800 4150
+	0    1    1    0
+$EndComp
 $EndSCHEMATC
