File: IO.sch (KiCad schematic (older format))
At the start: 13 parts

Commit message: sch updates
Parts:
- added J?: Conn_02x10_Odd_Even, symbol Connector_Generic:Conn_02x06_Odd_Even
Connections:
- wire segments 32 -> 40
Other:
- note removed: "X"
- moved on the sheet: J?
Changed lines of the file:
@@
 Text GLabel 4500 1450 2    50   Output ~ 0
 Baseband-OUT
-Text GLabel 4500 2250 2    50   Output ~ 0
-Signaling-OFFHOOK
 Wire Notes Line
 	3850 4800 3850 6350
@@
 	0    1    -1   0
 $EndComp
-Text GLabel 7350 1450 0    50   Input ~ 0
+Text GLabel 7350 1350 0    50   Input ~ 0
 Baseband-IN
-Text GLabel 7350 2150 0    50   Input ~ 0
-Signaling-RINGDOWN
 Text Notes 5300 850  0    50   ~ 0
 Crossover Cable Example
@@
 	0    -1   -1   0
 $EndComp
-Text GLabel 7350 1350 0    50   Output ~ 0
+Text GLabel 7350 1450 0    50   Output ~ 0
 Baseband-OUT
-Text GLabel 7350 2250 0    50   Output ~ 0
+Text GLabel 7350 2150 0    50   Output ~ 0
 Signaling-OFFHOOK
 $Comp
@@
 Text GLabel 4500 1350 2    50   Input ~ 0
 Baseband-IN
-Text GLabel 4500 2150 2    50   Input ~ 0
-Signaling-RINGDOWN
 Wire Notes Line
 	4250 2450 7600 2450
 Wire Notes Line
-	4250 950  7600 950
+	4250 900  7600 900
 Wire Notes Line
 	4250 1600 7600 1600
@@
 Wire Notes Line
 	4250 2450 4250 1750
-Text Notes 5850 1300 0    50   ~ 0
-X
-$Comp
-L power:GND #PWR?
-U 1 1 60ECC43D
-P 4500 2050
-AR Path="/60ECC43D" Ref="#PWR?"  Part="1"
-AR Path="/60E9D9E5/60ECC43D" Ref="#PWR?"  Part="1"
-F 0 "#PWR?" H 4500 1800 50  0001 C CNN
-F 1 "GND" V 4505 1922 50  0000 R CNN
-F 2 "" H 4500 2050 50  0001 C CNN
-F 3 "" H 4500 2050 50  0001 C CNN
-	1    4500 2050
-	0    -1   -1   0
-$EndComp
-$Comp
-L power:GND #PWR?
-U 1 1 60ECC77D
-P 7350 2050
-AR Path="/60ECC77D" Ref="#PWR?"  Part="1"
-AR Path="/60E9D9E5/60ECC77D" Ref="#PWR?"  Part="1"
-F 0 "#PWR?" H 7350 1800 50  0001 C CNN
-F 1 "GND" V 7355 1922 50  0000 R CNN
-F 2 "" H 7350 2050 50  0001 C CNN
-F 3 "" H 7350 2050 50  0001 C CNN
-	1    7350 2050
-	0    1    -1   0
-$EndComp
-Text Notes 5850 2250 0    50   ~ 0
-X
 $Comp
 L Connector_Generic:Conn_01x08 J?
@@
 L Connector:AudioPlug3 J?
 U 1 1 6101043E
-P 9800 4950
-F 0 "J?" H 9270 4904 50  0000 R CNN
-F 1 "AudioPlug3" H 9270 4995 50  0000 R CNN
-F 2 "" H 9900 4900 50  0001 C CNN
-F 3 "~" H 9900 4900 50  0001 C CNN
-	1    9800 4950
+P 9900 1300
+F 0 "J?" H 9370 1254 50  0000 R CNN
+F 1 "AudioPlug3" H 9370 1345 50  0000 R CNN
+F 2 "" H 10000 1250 50  0001 C CNN
+F 3 "~" H 10000 1250 50  0001 C CNN
+	1    9900 1300
 	-1   0    0    1
 $EndComp
@@
 L Connector:AudioPlug3 J?
 U 1 1 61011A7F
-P 9800 5750
-F 0 "J?" H 9270 5704 50  0000 R CNN
-F 1 "AudioPlug3" H 9270 5795 50  0000 R CNN
-F 2 "" H 9900 5700 50  0001 C CNN
-F 3 "~" H 9900 5700 50  0001 C CNN
-	1    9800 5750
+P 9900 2100
+F 0 "J?" H 9370 2054 50  0000 R CNN
+F 1 "AudioPlug3" H 9370 2145 50  0000 R CNN
+F 2 "" H 10000 2050 50  0001 C CNN
+F 3 "~" H 10000 2050 50  0001 C CNN
+	1    9900 2100
 	-1   0    0    1
 $EndComp
-Text Notes 8900 4400 0    50   ~ 0
+Text Notes 8850 700  0    50   ~ 0
 Kenwood 2-Pin
 Wire Notes Line
-	8650 4200 8650 6350
-Wire Notes Line
-	8650 6350 10900 6350
-Wire Notes Line
-	10900 6350 10900 4200
-Wire Notes Line
-	10900 4200 8650 4200
-Text GLabel 9200 4950 0    50   Input ~ 0
+	8750 550  8750 4300
+Wire Notes Line
+	8750 4300 11000 4300
+Wire Notes Line
+	11000 4300 11000 550
+Wire Notes Line
+	11000 550  8750 550
+Text GLabel 9300 1300 0    50   Input ~ 0
 KW-PROG
 $Comp
 L power:GND #PWR?
 U 1 1 61017F92
-P 9200 5050
+P 9300 1400
 AR Path="/61017F92" Ref="#PWR?"  Part="1"
 AR Path="/60E9D9E5/61017F92" Ref="#PWR?"  Part="1"
-F 0 "#PWR?" H 9200 4800 50  0001 C CNN
-F 1 "GND" V 9205 4922 50  0000 R CNN
-F 2 "" H 9200 5050 50  0001 C CNN
-F 3 "" H 9200 5050 50  0001 C CNN
-	1    9200 5050
+F 0 "#PWR?" H 9300 1150 50  0001 C CNN
+F 1 "GND" V 9305 1272 50  0000 R CNN
+F 2 "" H 9300 1400 50  0001 C CNN
+F 3 "" H 9300 1400 50  0001 C CNN
+	1    9300 1400
 	0    1    1    0
 $EndComp
@@
 L power:+5V #PWR?
 U 1 1 610186A8
-P 9200 5650
+P 9300 2000
 AR Path="/610186A8" Ref="#PWR?"  Part="1"
 AR Path="/60E9D9E5/610186A8" Ref="#PWR?"  Part="1"
-F 0 "#PWR?" H 9200 5500 50  0001 C CNN
-F 1 "+5V" V 9215 5778 50  0000 L CNN
-F 2 "" H 9200 5650 50  0001 C CNN
-F 3 "" H 9200 5650 50  0001 C CNN
-	1    9200 5650
-	0    -1   -1   0
-$EndComp
-Text Notes 9550 5500 0    50   ~ 0
+F 0 "#PWR?" H 9300 1850 50  0001 C CNN
+F 1 "+5V" V 9315 2128 50  0000 L CNN
+F 2 "" H 9300 2000 50  0001 C CNN
+F 3 "" H 9300 2000 50  0001 C CNN
+	1    9300 2000
+	0    -1   -1   0
+$EndComp
+Text Notes 9650 1850 0    50   ~ 0
 3.5mm
-Text Notes 9550 4700 0    50   ~ 0
+Text Notes 9650 1050 0    50   ~ 0
 2.5mm
-Text GLabel 9200 4850 0    50   Input ~ 0
+Text GLabel 9300 1200 0    50   Output ~ 0
 KW-SPK
-Text GLabel 9200 5750 0    50   Input ~ 0
+Text GLabel 9300 2100 0    50   Input ~ 0
 KW-MIC
-Text GLabel 9200 5850 0    50   Input ~ 0
+Text GLabel 9300 2200 0    50   Input ~ 0
 KW-PTT
+$Comp
+L power:+5V #PWR?
+U 1 1 610278AD
+P 7350 2250
+AR Path="/610278AD" Ref="#PWR?"  Part="1"
+AR Path="/60E9D9E5/610278AD" Ref="#PWR?"  Part="1"
+F 0 "#PWR?" H 7350 2100 50  0001 C CNN
+F 1 "+5V" V 7365 2378 50  0000 L CNN
+F 2 "" H 7350 2250 50  0001 C CNN
+F 3 "" H 7350 2250 50  0001 C CNN
+	1    7350 2250
+	0    -1   -1   0
+$EndComp
+$Comp
+L power:+5V #PWR?
+U 1 1 61028036
+P 4500 2250
+AR Path="/61028036" Ref="#PWR?"  Part="1"
+AR Path="/60E9D9E5/61028036" Ref="#PWR?"  Part="1"
+F 0 "#PWR?" H 4500 2100 50  0001 C CNN
+F 1 "+5V" V 4515 2378 50  0000 L CNN
+F 2 "" H 4500 2250 50  0001 C CNN
+F 3 "" H 4500 2250 50  0001 C CNN
+	1    4500 2250
+	0    1    1    0
+$EndComp
+Text GLabel 7350 2050 0    50   Input ~ 0
+Signaling-RINGDOWN
+Text GLabel 4500 2050 2    50   Input ~ 0
+Signaling-RINGDOWN
+Text GLabel 4500 2150 2    50   Output ~ 0
+Signaling-OFFHOOK
+Wire Wire Line
+	5400 2150 6450 2050
+Wire Wire Line
+	6450 2150 5400 2050
+Wire Wire Line
+	5400 1950 6450 1950
+Wire Wire Line
+	5400 2250 6450 2250
+Wire Wire Line
+	6500 1450 5350 1350
+Wire Wire Line
+	5350 1450 6500 1350
+Wire Wire Line
+	5350 1250 6500 1250
+Wire Wire Line
+	6500 1150 5350 1150
+$Comp
+L Connector_Generic:Conn_02x06_Odd_Even J?
+U 1 1 61037BFE
+P 9900 3450
+AR Path="/61037BFE" Ref="J?"  Part="1"
+AR Path="/60E9D9E5/61037BFE" Ref="J?"  Part="1"
+F 0 "J?" H 9950 4067 50  0000 C CNN
+F 1 "Conn_02x10_Odd_Even" H 9950 3976 50  0000 C CNN
+F 2 "" H 9900 3450 50  0001 C CNN
+F 3 "~" H 9900 3450 50  0001 C CNN
+	1    9900 3450
+	1    0    0    -1
+$EndComp
+Text GLabel 10200 3650 2    50   Input ~ 0
+KW-PROG
+Text GLabel 10200 3350 2    50   Output ~ 0
+KW-SPK
+Text GLabel 10200 3450 2    50   Input ~ 0
+KW-MIC
+Text GLabel 10200 3550 2    50   Input ~ 0
+KW-PTT
+$Comp
+L power:+5V #PWR?
+U 1 1 6103BBFB
+P 9700 3250
+AR Path="/6103BBFB" Ref="#PWR?"  Part="1"
+AR Path="/60E9D9E5/6103BBFB" Ref="#PWR?"  Part="1"
+F 0 "#PWR?" H 9700 3100 50  0001 C CNN
+F 1 "+5V" V 9715 3378 50  0000 L CNN
+F 2 "" H 9700 3250 50  0001 C CNN
+F 3 "" H 9700 3250 50  0001 C CNN
+	1    9700 3250
+	0    -1   -1   0
+$EndComp
+$Comp
+L power:GND #PWR?
+U 1 1 6103C4E0
+P 10200 3750
+AR Path="/6103C4E0" Ref="#PWR?"  Part="1"
+AR Path="/60E9D9E5/6103C4E0" Ref="#PWR?"  Part="1"
+F 0 "#PWR?" H 10200 3500 50  0001 C CNN
+F 1 "GND" V 10205 3622 50  0000 R CNN
+F 2 "" H 10200 3750 50  0001 C CNN
+F 3 "" H 10200 3750 50  0001 C CNN
+	1    10200 3750
+	0    -1   -1   0
+$EndComp
+Text GLabel 9700 3450 0    50   Input ~ 0
+Baseband-IN
+Text GLabel 9700 3350 0    50   Output ~ 0
+Baseband-OUT
+Text GLabel 9700 3550 0    50   Output ~ 0
+Signaling-OFFHOOK
+Text GLabel 9700 3650 0    50   Input ~ 0
+Signaling-RINGDOWN
+$Comp
+L power:GND #PWR?
+U 1 1 61049B14
+P 9700 3750
+AR Path="/61049B14" Ref="#PWR?"  Part="1"
+AR Path="/60E9D9E5/61049B14" Ref="#PWR?"  Part="1"
+F 0 "#PWR?" H 9700 3500 50  0001 C CNN
+F 1 "GND" V 9705 3622 50  0000 R CNN
+F 2 "" H 9700 3750 50  0001 C CNN
+F 3 "" H 9700 3750 50  0001 C CNN
+	1    9700 3750
+	0    1    1    0
+$EndComp
+$Comp
+L power:+5V #PWR?
+U 1 1 6104A832
+P 10200 3250
+AR Path="/6104A832" Ref="#PWR?"  Part="1"
+AR Path="/60E9D9E5/6104A832" Ref="#PWR?"  Part="1"
+F 0 "#PWR?" H 10200 3100 50  0001 C CNN
+F 1 "+5V" V 10215 3378 50  0000 L CNN
+F 2 "" H 10200 3250 50  0001 C CNN
+F 3 "" H 10200 3250 50  0001 C CNN
+	1    10200 3250
+	0    1    1    0
+$EndComp
+Wire Notes Line
+	9550 2400 9400 2400
+Wire Notes Line
+	9400 2400 9400 1000
+Wire Notes Line
+	9400 1000 9550 1000
+Wire Notes Line
+	9550 1000 9550 2400
 $EndSCHEMATC

Commit message: updates
Parts:
- added J?: Conn_01x08_Male, symbol Connector_Generic:Conn_01x08
Other:
- note added: "RJ45 E&M Pinout\n"
- note added: "RJ45 Expansion Interface\n"
- note removed: "E&M Type Output interface"
- note removed: "RJ45 Module Interface\nTELEPHONY"
Changed lines of the file:
@@
 	1    0    0    1
 $EndComp
-Text Notes 3900 6300 0    50   ~ 0
-E&M Type Output interface
 $Comp
 L Connector:RJ45 J?
@@
 $EndComp
 Text Notes 5050 5650 0    50   ~ 0
-RJ45 Module Interface\nTELEPHONY
+RJ45 Expansion Interface\n
 Text GLabel 7050 3250 2    50   Output ~ 0
 RST_Request
@@
 	1    0    0    -1
 $EndComp
-Text GLabel 4000 5900 2    50   Input ~ 0
+Text GLabel 9750 5900 2    50   Input ~ 0
 E&M-SB
-Text GLabel 4000 5200 2    50   Input ~ 0
+Text GLabel 9750 5200 2    50   Input ~ 0
 E&M-SG
-Text GLabel 4000 5800 2    50   Input ~ 0
+Text GLabel 9750 5800 2    50   Input ~ 0
 E&M-M
-Text GLabel 4000 5400 2    50   Input ~ 0
+Text GLabel 9750 5400 2    50   Input ~ 0
 E&M-T1
-Text GLabel 4000 5300 2    50   Input ~ 0
+Text GLabel 9750 5300 2    50   Input ~ 0
 E&M-E
-Text GLabel 4000 5700 2    50   Input ~ 0
+Text GLabel 9750 5700 2    50   Input ~ 0
 E&M-R1
-Text GLabel 4000 5600 2    50   Input ~ 0
+Text GLabel 9750 5600 2    50   Input ~ 0
 E&M-R
-Text GLabel 4000 5500 2    50   Input ~ 0
+Text GLabel 9750 5500 2    50   Input ~ 0
 E&M-T
 Wire Wire Line
@@
 Kenwood 2-Pin
 Wire Notes Line
-	8750 550  8750 4300
-Wire Notes Line
-	8750 4300 11000 4300
-Wire Notes Line
-	11000 4300 11000 550
+	8750 550  8750 4500
+Wire Notes Line
+	8750 4500 11000 4500
+Wire Notes Line
+	11000 4500 11000 550
 Wire Notes Line
 	11000 550  8750 550
@@
 Wire Notes Line
 	9550 1000 9550 2400
+$Comp
+L Connector_Generic:Conn_01x08 J?
+U 1 1 60FD1319
+P 9550 5600
+AR Path="/60FD1319" Ref="J?"  Part="1"
+AR Path="/60E9D9E5/60FD1319" Ref="J?"  Part="1"
+F 0 "J?" H 9468 4975 50  0000 C CNN
+F 1 "Conn_01x08_Male" H 9468 5066 50  0000 C CNN
+F 2 "" H 9550 5600 50  0001 C CNN
+F 3 "~" H 9550 5600 50  0001 C CNN
+	1    9550 5600
+	-1   0    0    1
+$EndComp
+Text Notes 8850 6250 0    50   ~ 0
+RJ45 E&M Pinout\n
+Wire Notes Line
+	8750 4800 8750 6350
+Wire Notes Line
+	8750 6350 11000 6350
+Wire Notes Line
+	11000 6350 11000 4800
+Wire Notes Line
+	11000 4800 8750 4800
 $EndSCHEMATC
