File: uController.sch (KiCad schematic (older format))
At the start: 17 parts

Commit message: more updates
Connections:
- wire segments 33 -> 34
Other:
- note added: "TEST Reset Circuit n-mos?\n"
- note removed: "TEST Reset Circuit"
- moved on the sheet: J?, R?, SW?
Changed lines of the file:
@@
 L Switch:SW_Push SW?
 U 1 1 60E968E0
-P 9900 1450
+P 2950 5000
 AR Path="/60E968E0" Ref="SW?"  Part="1"
 AR Path="/60E76DCE/60E968E0" Ref="SW?"  Part="1"
-F 0 "SW?" H 9900 1735 50  0000 C CNN
-F 1 "SW_Push" H 9900 1644 50  0000 C CNN
-F 2 "" H 9900 1650 50  0001 C CNN
-F 3 "~" H 9900 1650 50  0001 C CNN
-	1    9900 1450
-	1    0    0    -1
-$EndComp
-Text GLabel 9050 1450 0    50   Input ~ 0
+F 0 "SW?" H 2950 5285 50  0000 C CNN
+F 1 "SW_Push" H 2950 5194 50  0000 C CNN
+F 2 "" H 2950 5200 50  0001 C CNN
+F 3 "~" H 2950 5200 50  0001 C CNN
+	1    2950 5000
+	1    0    0    -1
+$EndComp
+Text GLabel 2100 5000 0    50   Input ~ 0
 Mega-nRST
 $Comp
 L Device:R R?
 U 1 1 60E968E7
-P 9500 1600
+P 2550 4650
 AR Path="/60E968E7" Ref="R?"  Part="1"
 AR Path="/60E76DCE/60E968E7" Ref="R?"  Part="1"
-F 0 "R?" H 9430 1554 50  0000 R CNN
-F 1 "1K" H 9430 1645 50  0000 R CNN
-F 2 "" V 9430 1600 50  0001 C CNN
-F 3 "~" H 9500 1600 50  0001 C CNN
-	1    9500 1600
+F 0 "R?" H 2480 4604 50  0000 R CNN
+F 1 "1K" H 2480 4695 50  0000 R CNN
+F 2 "" V 2480 4650 50  0001 C CNN
+F 3 "~" H 2550 4650 50  0001 C CNN
+	1    2550 4650
 	-1   0    0    1
 $EndComp
-Text Notes 8500 1250 0    50   ~ 0
+Text Notes 1550 4800 0    50   ~ 0
 Reset (Pullup)
 Text GLabel 8900 3550 0    50   Input ~ 0
@@
 Text Notes 8350 3800 0    50   ~ 0
 CLOCK
-Text Notes 1450 3150 0    50   ~ 0
+Text Notes 1000 1000 0    50   ~ 0
 ICSP
 $Comp
@@
 L Connector_Generic:Conn_02x03_Odd_Even J?
 U 1 1 60E96908
-P 2150 3450
+P 1700 1300
 AR Path="/60E96908" Ref="J?"  Part="1"
 AR Path="/60E76DCE/60E96908" Ref="J?"  Part="1"
-F 0 "J?" H 2200 3767 50  0000 C CNN
-F 1 "Conn_02x03_Odd_Even" H 2200 3676 50  0000 C CNN
-F 2 "" H 2150 3450 50  0001 C CNN
-F 3 "~" H 2150 3450 50  0001 C CNN
-	1    2150 3450
+F 0 "J?" H 1750 1617 50  0000 C CNN
+F 1 "Conn_02x03_Odd_Even" H 1750 1526 50  0000 C CNN
+F 2 "" H 1700 1300 50  0001 C CNN
+F 3 "~" H 1700 1300 50  0001 C CNN
+	1    1700 1300
 	1    0    0    -1
 $EndComp
@@
 L power:GND #PWR?
 U 1 1 60E9690E
-P 2450 3550
+P 2000 1400
 AR Path="/60E9690E" Ref="#PWR?"  Part="1"
 AR Path="/60E76DCE/60E9690E" Ref="#PWR?"  Part="1"
-F 0 "#PWR?" H 2450 3300 50  0001 C CNN
-F 1 "GND" V 2455 3422 50  0000 R CNN
-F 2 "" H 2450 3550 50  0001 C CNN
-F 3 "" H 2450 3550 50  0001 C CNN
-	1    2450 3550
+F 0 "#PWR?" H 2000 1150 50  0001 C CNN
+F 1 "GND" V 2005 1272 50  0000 R CNN
+F 2 "" H 2000 1400 50  0001 C CNN
+F 3 "" H 2000 1400 50  0001 C CNN
+	1    2000 1400
 	0    -1   -1   0
 $EndComp
@@
 L power:+5V #PWR?
 U 1 1 60E96914
-P 2450 3350
+P 2000 1200
 AR Path="/60E96914" Ref="#PWR?"  Part="1"
 AR Path="/60E76DCE/60E96914" Ref="#PWR?"  Part="1"
-F 0 "#PWR?" H 2450 3200 50  0001 C CNN
-F 1 "+5V" V 2465 3478 50  0000 L CNN
-F 2 "" H 2450 3350 50  0001 C CNN
-F 3 "" H 2450 3350 50  0001 C CNN
-	1    2450 3350
-	0    1    1    0
-$EndComp
-Text GLabel 2450 3450 2    50   Input ~ 0
+F 0 "#PWR?" H 2000 1050 50  0001 C CNN
+F 1 "+5V" V 2015 1328 50  0000 L CNN
+F 2 "" H 2000 1200 50  0001 C CNN
+F 3 "" H 2000 1200 50  0001 C CNN
+	1    2000 1200
+	0    1    1    0
+$EndComp
+Text GLabel 2000 1300 2    50   Input ~ 0
 Mega-PB3
-Text GLabel 1950 3550 0    50   Input ~ 0
+Text GLabel 1500 1400 0    50   Input ~ 0
 Mega-RST
-Text GLabel 1950 3450 0    50   Input ~ 0
+Text GLabel 1500 1300 0    50   Input ~ 0
 Mega-PB5
-Text GLabel 1950 3350 0    50   Input ~ 0
+Text GLabel 1500 1200 0    50   Input ~ 0
 Mega-PB4
 $Comp
 L power:+5V #PWR?
 U 1 1 60E9691E
-P 9500 1750
+P 2550 4500
 AR Path="/60E9691E" Ref="#PWR?"  Part="1"
 AR Path="/60E76DCE/60E9691E" Ref="#PWR?"  Part="1"
-F 0 "#PWR?" H 9500 1600 50  0001 C CNN
-F 1 "+5V" H 9515 1923 50  0000 C CNN
-F 2 "" H 9500 1750 50  0001 C CNN
-F 3 "" H 9500 1750 50  0001 C CNN
-	1    9500 1750
-	-1   0    0    1
+F 0 "#PWR?" H 2550 4350 50  0001 C CNN
+F 1 "+5V" H 2565 4673 50  0000 C CNN
+F 2 "" H 2550 4500 50  0001 C CNN
+F 3 "" H 2550 4500 50  0001 C CNN
+	1    2550 4500
+	1    0    0    -1
 $EndComp
 $Comp
 L power:GND #PWR?
 U 1 1 60E96924
-P 10350 1750
+P 3400 5150
 AR Path="/60E96924" Ref="#PWR?"  Part="1"
 AR Path="/60E76DCE/60E96924" Ref="#PWR?"  Part="1"
-F 0 "#PWR?" H 10350 1500 50  0001 C CNN
-F 1 "GND" V 10355 1622 50  0000 R CNN
-F 2 "" H 10350 1750 50  0001 C CNN
-F 3 "" H 10350 1750 50  0001 C CNN
-	1    10350 1750
-	1    0    0    -1
-$EndComp
-Wire Wire Line
-	9500 1450 9050 1450
-Wire Wire Line
-	9700 1450 9500 1450
-Connection ~ 9500 1450
+F 0 "#PWR?" H 3400 4900 50  0001 C CNN
+F 1 "GND" V 3405 5022 50  0000 R CNN
+F 2 "" H 3400 5150 50  0001 C CNN
+F 3 "" H 3400 5150 50  0001 C CNN
+	1    3400 5150
+	1    0    0    -1
+$EndComp
 Wire Wire Line
 	9750 3550 9300 3550
@@
 	10050 3950 10350 3950
 Wire Wire Line
-	10350 1750 10350 1450
-Wire Wire Line
-	10100 1450 10350 1450
+	3400 5150 3400 5000
+Wire Wire Line
+	3150 5000 3400 5000
 $Comp
 L Switch:SW_Push SW?
@@
 	1900 6100 2450 6100
 Text Notes 1000 5850 0    50   ~ 0
-TEST Reset Circuit
+TEST Reset Circuit n-mos?\n
 Wire Notes Line
 	900  5650 900  7100
@@
 Wire Notes Line
 	4200 5650 900  5650
+Wire Wire Line
+	2100 5000 2550 5000
+Wire Wire Line
+	2550 4800 2550 5000
+Connection ~ 2550 5000
+Wire Wire Line
+	2550 5000 2750 5000
 $EndSCHEMATC

Commit message: updates
Other:
- moved on the sheet: R?, SW?
Changed lines of the file:
@@
 $Descr A4 11693 8268
 encoding utf-8
-Sheet 4 10
+Sheet 4 11
 Title "300 Baud Audio FSK Modem "
 Date "2021-07-08"
@@
 L Switch:SW_Push SW?
 U 1 1 60E968E0
-P 2950 5000
+P 2600 4150
 AR Path="/60E968E0" Ref="SW?"  Part="1"
 AR Path="/60E76DCE/60E968E0" Ref="SW?"  Part="1"
-F 0 "SW?" H 2950 5285 50  0000 C CNN
-F 1 "SW_Push" H 2950 5194 50  0000 C CNN
-F 2 "" H 2950 5200 50  0001 C CNN
-F 3 "~" H 2950 5200 50  0001 C CNN
-	1    2950 5000
-	1    0    0    -1
-$EndComp
-Text GLabel 2100 5000 0    50   Input ~ 0
+F 0 "SW?" H 2600 4435 50  0000 C CNN
+F 1 "SW_Push" H 2600 4344 50  0000 C CNN
+F 2 "" H 2600 4350 50  0001 C CNN
+F 3 "~" H 2600 4350 50  0001 C CNN
+	1    2600 4150
+	1    0    0    -1
+$EndComp
+Text GLabel 1750 4150 0    50   Input ~ 0
 Mega-nRST
 $Comp
 L Device:R R?
 U 1 1 60E968E7
-P 2550 4650
+P 2200 3800
 AR Path="/60E968E7" Ref="R?"  Part="1"
 AR Path="/60E76DCE/60E968E7" Ref="R?"  Part="1"
-F 0 "R?" H 2480 4604 50  0000 R CNN
-F 1 "1K" H 2480 4695 50  0000 R CNN
-F 2 "" V 2480 4650 50  0001 C CNN
-F 3 "~" H 2550 4650 50  0001 C CNN
-	1    2550 4650
+F 0 "R?" H 2130 3754 50  0000 R CNN
+F 1 "1K" H 2130 3845 50  0000 R CNN
+F 2 "" V 2130 3800 50  0001 C CNN
+F 3 "~" H 2200 3800 50  0001 C CNN
+	1    2200 3800
 	-1   0    0    1
 $EndComp
-Text Notes 1550 4800 0    50   ~ 0
+Text Notes 1200 3950 0    50   ~ 0
 Reset (Pullup)
 Text GLabel 8900 3550 0    50   Input ~ 0
@@
 L power:+5V #PWR?
 U 1 1 60E9691E
-P 2550 4500
+P 2200 3650
 AR Path="/60E9691E" Ref="#PWR?"  Part="1"
 AR Path="/60E76DCE/60E9691E" Ref="#PWR?"  Part="1"
-F 0 "#PWR?" H 2550 4350 50  0001 C CNN
-F 1 "+5V" H 2565 4673 50  0000 C CNN
-F 2 "" H 2550 4500 50  0001 C CNN
-F 3 "" H 2550 4500 50  0001 C CNN
-	1    2550 4500
+F 0 "#PWR?" H 2200 3500 50  0001 C CNN
+F 1 "+5V" H 2215 3823 50  0000 C CNN
+F 2 "" H 2200 3650 50  0001 C CNN
+F 3 "" H 2200 3650 50  0001 C CNN
+	1    2200 3650
 	1    0    0    -1
 $EndComp
@@
 L power:GND #PWR?
 U 1 1 60E96924
-P 3400 5150
+P 3050 4300
 AR Path="/60E96924" Ref="#PWR?"  Part="1"
 AR Path="/60E76DCE/60E96924" Ref="#PWR?"  Part="1"
-F 0 "#PWR?" H 3400 4900 50  0001 C CNN
-F 1 "GND" V 3405 5022 50  0000 R CNN
-F 2 "" H 3400 5150 50  0001 C CNN
-F 3 "" H 3400 5150 50  0001 C CNN
-	1    3400 5150
+F 0 "#PWR?" H 3050 4050 50  0001 C CNN
+F 1 "GND" V 3055 4172 50  0000 R CNN
+F 2 "" H 3050 4300 50  0001 C CNN
+F 3 "" H 3050 4300 50  0001 C CNN
+	1    3050 4300
 	1    0    0    -1
 $EndComp
@@
 	10050 3950 10350 3950
 Wire Wire Line
-	3400 5150 3400 5000
-Wire Wire Line
-	3150 5000 3400 5000
+	3050 4300 3050 4150
+Wire Wire Line
+	2800 4150 3050 4150
 $Comp
 L Switch:SW_Push SW?
@@
 	4200 5650 900  5650
 Wire Wire Line
-	2100 5000 2550 5000
-Wire Wire Line
-	2550 4800 2550 5000
-Connection ~ 2550 5000
-Wire Wire Line
-	2550 5000 2750 5000
+	1750 4150 2200 4150
+Wire Wire Line
+	2200 3950 2200 4150
+Connection ~ 2200 4150
+Wire Wire Line
+	2200 4150 2400 4150
 $EndSCHEMATC

Commit message: updates
Other:
- moved on the sheet: J?
Changed lines of the file:
@@
 Text Notes 8350 3800 0    50   ~ 0
 CLOCK
-Text Notes 1000 1000 0    50   ~ 0
+Text Notes 8500 1000 0    50   ~ 0
 ICSP
 $Comp
@@
 L Connector_Generic:Conn_02x03_Odd_Even J?
 U 1 1 60E96908
-P 1700 1300
+P 9200 1300
 AR Path="/60E96908" Ref="J?"  Part="1"
 AR Path="/60E76DCE/60E96908" Ref="J?"  Part="1"
-F 0 "J?" H 1750 1617 50  0000 C CNN
-F 1 "Conn_02x03_Odd_Even" H 1750 1526 50  0000 C CNN
-F 2 "" H 1700 1300 50  0001 C CNN
-F 3 "~" H 1700 1300 50  0001 C CNN
-	1    1700 1300
+F 0 "J?" H 9250 1617 50  0000 C CNN
+F 1 "Conn_02x03_Odd_Even" H 9250 1526 50  0000 C CNN
+F 2 "" H 9200 1300 50  0001 C CNN
+F 3 "~" H 9200 1300 50  0001 C CNN
+	1    9200 1300
 	1    0    0    -1
 $EndComp
@@
 L power:GND #PWR?
 U 1 1 60E9690E
-P 2000 1400
+P 9500 1400
 AR Path="/60E9690E" Ref="#PWR?"  Part="1"
 AR Path="/60E76DCE/60E9690E" Ref="#PWR?"  Part="1"
-F 0 "#PWR?" H 2000 1150 50  0001 C CNN
-F 1 "GND" V 2005 1272 50  0000 R CNN
-F 2 "" H 2000 1400 50  0001 C CNN
-F 3 "" H 2000 1400 50  0001 C CNN
-	1    2000 1400
+F 0 "#PWR?" H 9500 1150 50  0001 C CNN
+F 1 "GND" V 9505 1272 50  0000 R CNN
+F 2 "" H 9500 1400 50  0001 C CNN
+F 3 "" H 9500 1400 50  0001 C CNN
+	1    9500 1400
 	0    -1   -1   0
 $EndComp
@@
 L power:+5V #PWR?
 U 1 1 60E96914
-P 2000 1200
+P 9500 1200
 AR Path="/60E96914" Ref="#PWR?"  Part="1"
 AR Path="/60E76DCE/60E96914" Ref="#PWR?"  Part="1"
-F 0 "#PWR?" H 2000 1050 50  0001 C CNN
-F 1 "+5V" V 2015 1328 50  0000 L CNN
-F 2 "" H 2000 1200 50  0001 C CNN
-F 3 "" H 2000 1200 50  0001 C CNN
-	1    2000 1200
+F 0 "#PWR?" H 9500 1050 50  0001 C CNN
+F 1 "+5V" V 9515 1328 50  0000 L CNN
+F 2 "" H 9500 1200 50  0001 C CNN
+F 3 "" H 9500 1200 50  0001 C CNN
+	1    9500 1200
 	0    1    1    0
 $EndComp
-Text GLabel 2000 1300 2    50   Input ~ 0
+Text GLabel 9500 1300 2    50   Input ~ 0
 Mega-PB3
-Text GLabel 1500 1400 0    50   Input ~ 0
+Text GLabel 9000 1400 0    50   Input ~ 0
 Mega-RST
-Text GLabel 1500 1300 0    50   Input ~ 0
+Text GLabel 9000 1300 0    50   Input ~ 0
 Mega-PB5
-Text GLabel 1500 1200 0    50   Input ~ 0
+Text GLabel 9000 1200 0    50   Input ~ 0
 Mega-PB4
 $Comp

Commit message: fixed reset circuit
Parts:
- removed C?: 100u, symbol Device:C_Polarized
- removed Q?: Q_PMOS_SDG, symbol Device:Q_PMOS_SDG
- removed R?: 220, symbol Device:R
- removed R?: 10K, symbol Device:R
- removed SW?: SW_Push, symbol Switch:SW_Push
- removed U?: 74LS14, symbol 74xx:74LS14
- added Q?: Q_NMOS_DGS, symbol Device:Q_NMOS_DGS
- added R? (x2): 1K, symbol Device:R
Connections:
- wire segments 34 -> 35
Other:
- note added: "Reset Circuit with digital select via p-mos select\n"
- note removed: "TEST Reset Circuit n-mos?\n"
- moved on the sheet: R?, SW?
Changed lines of the file:
@@
 Text GLabel 6150 4800 2    50   Input ~ 0
 TTL-RX
-Text GLabel 6150 5850 2    50   Input ~ 0
+Text GLabel 6150 5800 2    50   Input ~ 0
 TTL-DCD
 Text GLabel 6150 5000 2    50   Input ~ 0
@@
 L Switch:SW_Push SW?
 U 1 1 60E968E0
-P 2600 4150
+P 2000 6600
 AR Path="/60E968E0" Ref="SW?"  Part="1"
 AR Path="/60E76DCE/60E968E0" Ref="SW?"  Part="1"
-F 0 "SW?" H 2600 4435 50  0000 C CNN
-F 1 "SW_Push" H 2600 4344 50  0000 C CNN
-F 2 "" H 2600 4350 50  0001 C CNN
-F 3 "~" H 2600 4350 50  0001 C CNN
-	1    2600 4150
+F 0 "SW?" H 2000 6885 50  0000 C CNN
+F 1 "SW_Push" H 2000 6794 50  0000 C CNN
+F 2 "" H 2000 6800 50  0001 C CNN
+F 3 "~" H 2000 6800 50  0001 C CNN
+	1    2000 6600
 	1    0    0    -1
 $EndComp
-Text GLabel 1750 4150 0    50   Input ~ 0
+Text GLabel 1300 6600 0    50   Input ~ 0
 Mega-nRST
 $Comp
 L Device:R R?
 U 1 1 60E968E7
-P 2200 3800
+P 1250 7100
 AR Path="/60E968E7" Ref="R?"  Part="1"
 AR Path="/60E76DCE/60E968E7" Ref="R?"  Part="1"
-F 0 "R?" H 2130 3754 50  0000 R CNN
-F 1 "1K" H 2130 3845 50  0000 R CNN
-F 2 "" V 2130 3800 50  0001 C CNN
-F 3 "~" H 2200 3800 50  0001 C CNN
-	1    2200 3800
-	-1   0    0    1
-$EndComp
-Text Notes 1200 3950 0    50   ~ 0
+F 0 "R?" H 1180 7054 50  0000 R CNN
+F 1 "1K" H 1180 7145 50  0000 R CNN
+F 2 "" V 1180 7100 50  0001 C CNN
+F 3 "~" H 1250 7100 50  0001 C CNN
+	1    1250 7100
+	0    1    1    0
+$EndComp
+Text Notes 700  6450 0    50   ~ 0
 Reset (Pullup)
 Text GLabel 8900 3550 0    50   Input ~ 0
@@
 Text GLabel 8900 3950 0    50   Input ~ 0
 Mega-XTAL2
-Text Notes 8350 3800 0    50   ~ 0
+Text Notes 8300 3300 0    50   ~ 0
 CLOCK
 Text Notes 8500 1000 0    50   ~ 0
@@
 L power:+5V #PWR?
 U 1 1 60E9691E
-P 2200 3650
+P 1100 7100
 AR Path="/60E9691E" Ref="#PWR?"  Part="1"
 AR Path="/60E76DCE/60E9691E" Ref="#PWR?"  Part="1"
-F 0 "#PWR?" H 2200 3500 50  0001 C CNN
-F 1 "+5V" H 2215 3823 50  0000 C CNN
-F 2 "" H 2200 3650 50  0001 C CNN
-F 3 "" H 2200 3650 50  0001 C CNN
-	1    2200 3650
-	1    0    0    -1
+F 0 "#PWR?" H 1100 6950 50  0001 C CNN
+F 1 "+5V" H 1115 7273 50  0000 C CNN
+F 2 "" H 1100 7100 50  0001 C CNN
+F 3 "" H 1100 7100 50  0001 C CNN
+	1    1100 7100
+	0    -1   -1   0
 $EndComp
 $Comp
 L power:GND #PWR?
 U 1 1 60E96924
-P 3050 4300
+P 2650 6600
 AR Path="/60E96924" Ref="#PWR?"  Part="1"
 AR Path="/60E76DCE/60E96924" Ref="#PWR?"  Part="1"
-F 0 "#PWR?" H 3050 4050 50  0001 C CNN
-F 1 "GND" V 3055 4172 50  0000 R CNN
-F 2 "" H 3050 4300 50  0001 C CNN
-F 3 "" H 3050 4300 50  0001 C CNN
-	1    3050 4300
-	1    0    0    -1
+F 0 "#PWR?" H 2650 6350 50  0001 C CNN
+F 1 "GND" V 2655 6472 50  0000 R CNN
+F 2 "" H 2650 6600 50  0001 C CNN
+F 3 "" H 2650 6600 50  0001 C CNN
+	1    2650 6600
+	0    -1   -1   0
 $EndComp
 Wire Wire Line
@@
 	10050 3950 10350 3950
 Wire Wire Line
-	3050 4300 3050 4150
-Wire Wire Line
-	2800 4150 3050 4150
-$Comp
-L Switch:SW_Push SW?
-U 1 1 60EC9F93
-P 2950 6100
-AR Path="/60EC9F93" Ref="SW?"  Part="1"
-AR Path="/60E76DCE/60EC9F93" Ref="SW?"  Part="1"
-F 0 "SW?" H 2950 6385 50  0000 C CNN
-F 1 "SW_Push" H 2950 6294 50  0000 C CNN
-F 2 "" H 2950 6300 50  0001 C CNN
-F 3 "~" H 2950 6300 50  0001 C CNN
-	1    2950 6100
-	1    0    0    -1
-$EndComp
-$Comp
-L Device:C_Polarized C?
-U 1 1 60EC9F99
-P 3550 6100
-AR Path="/60EC9F99" Ref="C?"  Part="1"
-AR Path="/60E76DCE/60EC9F99" Ref="C?"  Part="1"
-F 0 "C?" V 3295 6100 50  0000 C CNN
-F 1 "100u" V 3386 6100 50  0000 C CNN
-F 2 "" H 3588 5950 50  0001 C CNN
-F 3 "~" H 3550 6100 50  0001 C CNN
-	1    3550 6100
-	0    1    1    0
-$EndComp
-Text GLabel 1900 6100 0    50   Input ~ 0
-Mega-nRST
-$Comp
-L power:+5V #PWR?
-U 1 1 60EC9FA0
-P 3700 6100
-AR Path="/60EC9FA0" Ref="#PWR?"  Part="1"
-AR Path="/60E76DCE/60EC9FA0" Ref="#PWR?"  Part="1"
-F 0 "#PWR?" H 3700 5950 50  0001 C CNN
-F 1 "+5V" V 3715 6228 50  0000 L CNN
-F 2 "" H 3700 6100 50  0001 C CNN
-F 3 "" H 3700 6100 50  0001 C CNN
-	1    3700 6100
-	0    1    1    0
-$EndComp
+	2200 6600 2450 6600
+Wire Wire Line
+	1400 7100 1600 7100
+Connection ~ 1600 6600
+Wire Wire Line
+	1600 6600 1800 6600
+Wire Wire Line
+	1600 6600 1600 7100
+Text GLabel 1300 7400 0    50   Input ~ 0
+RST_Request
+Wire Wire Line
+	2450 6600 2450 7100
+Wire Wire Line
+	1600 7100 1800 7100
+Text Notes 850  5750 0    50   ~ 0
+Reset Circuit with digital select via p-mos select\n
+Wire Wire Line
+	2650 6600 2450 6600
+Connection ~ 2450 6600
 $Comp
 L Device:R R?
-U 1 1 60EC9FA6
-P 2600 6100
-AR Path="/60EC9FA6" Ref="R?"  Part="1"
-AR Path="/60E76DCE/60EC9FA6" Ref="R?"  Part="1"
-F 0 "R?" V 2393 6100 50  0000 C CNN
-F 1 "220" V 2484 6100 50  0000 C CNN
-F 2 "" V 2530 6100 50  0001 C CNN
-F 3 "~" H 2600 6100 50  0001 C CNN
-	1    2600 6100
-	0    1    1    0
-$EndComp
+U 1 1 60EC31D3
+P 1750 7400
+AR Path="/60EC31D3" Ref="R?"  Part="1"
+AR Path="/60E76DCE/60EC31D3" Ref="R?"  Part="1"
+F 0 "R?" H 1680 7354 50  0000 R CNN
+F 1 "1K" H 1680 7445 50  0000 R CNN
+F 2 "" V 1680 7400 50  0001 C CNN
+F 3 "~" H 1750 7400 50  0001 C CNN
+	1    1750 7400
+	0    -1   -1   0
+$EndComp
+Wire Wire Line
+	2200 7100 2450 7100
 $Comp
 L Device:R R?
-U 1 1 60EC9FAC
-P 3400 6700
-AR Path="/60EC9FAC" Ref="R?"  Part="1"
-AR Path="/60E76DCE/60EC9FAC" Ref="R?"  Part="1"
-F 0 "R?" H 3330 6654 50  0000 R CNN
-F 1 "10K" H 3330 6745 50  0000 R CNN
-F 2 "" V 3330 6700 50  0001 C CNN
-F 3 "~" H 3400 6700 50  0001 C CNN
-	1    3400 6700
-	-1   0    0    1
-$EndComp
-$Comp
-L Device:Q_PMOS_SDG Q?
-U 1 1 60EC9FB2
-P 2950 6650
-AR Path="/60EC9FB2" Ref="Q?"  Part="1"
-AR Path="/60E76DCE/60EC9FB2" Ref="Q?"  Part="1"
-F 0 "Q?" V 3292 6650 50  0000 C CNN
-F 1 "Q_PMOS_SDG" V 3201 6650 50  0000 C CNN
-F 2 "" H 3150 6750 50  0001 C CNN
-F 3 "~" H 2950 6650 50  0001 C CNN
-	1    2950 6650
-	0    -1   -1   0
-$EndComp
-Wire Wire Line
-	3400 6550 3400 6100
-Wire Wire Line
-	2950 6850 2500 6850
-Connection ~ 2950 6850
-Wire Wire Line
-	3150 6550 3150 6100
-$Comp
-L 74xx:74LS14 U?
-U 1 1 60EC9FBC
-P 2200 6850
-AR Path="/60EC9FBC" Ref="U?"  Part="1"
-AR Path="/60E76DCE/60EC9FBC" Ref="U?"  Part="1"
-F 0 "U?" H 2200 7167 50  0000 C CNN
-F 1 "74LS14" H 2200 7076 50  0000 C CNN
-F 2 "" H 2200 6850 50  0001 C CNN
-F 3 "http://www.ti.com/lit/gpn/sn74LS14" H 2200 6850 50  0001 C CNN
-	1    2200 6850
-	1    0    0    -1
-$EndComp
-Wire Wire Line
-	2950 6850 3400 6850
-Wire Wire Line
-	3150 6100 3400 6100
-Connection ~ 3150 6100
-Connection ~ 3400 6100
-Text GLabel 1900 6850 0    50   Input ~ 0
-RST_Request
-Wire Wire Line
-	2750 6550 2750 6100
-Connection ~ 2750 6100
-Wire Wire Line
-	1900 6100 2450 6100
-Text Notes 1000 5850 0    50   ~ 0
-TEST Reset Circuit n-mos?\n
-Wire Notes Line
-	900  5650 900  7100
-Wire Notes Line
-	900  7100 4200 7100
-Wire Notes Line
-	4200 7100 4200 5650
-Wire Notes Line
-	4200 5650 900  5650
-Wire Wire Line
-	1750 4150 2200 4150
-Wire Wire Line
-	2200 3950 2200 4150
-Connection ~ 2200 4150
-Wire Wire Line
-	2200 4150 2400 4150
+U 1 1 60EC4332
+P 2300 7400
+AR Path="/60EC4332" Ref="R?"  Part="1"
+AR Path="/60E76DCE/60EC4332" Ref="R?"  Part="1"
+F 0 "R?" H 2230 7354 50  0000 R CNN
+F 1 "1K" H 2230 7445 50  0000 R CNN
+F 2 "" V 2230 7400 50  0001 C CNN
+F 3 "~" H 2300 7400 50  0001 C CNN
+	1    2300 7400
+	0    -1   -1   0
+$EndComp
+Wire Wire Line
+	2450 7100 2450 7400
+Connection ~ 2450 7100
+Wire Wire Line
+	1900 7400 2000 7400
+$Comp
+L Device:Q_NMOS_DGS Q?
+U 1 1 60ECA576
+P 2000 7200
+F 0 "Q?" V 2342 7200 50  0000 C CNN
+F 1 "Q_NMOS_DGS" V 2251 7200 50  0000 C CNN
+F 2 "" H 2200 7300 50  0001 C CNN
+F 3 "~" H 2000 7200 50  0001 C CNN
+	1    2000 7200
+	0    -1   -1   0
+$EndComp
+Connection ~ 2000 7400
+Wire Wire Line
+	2000 7400 2150 7400
+Wire Wire Line
+	1600 6600 1300 6600
+Wire Wire Line
+	1600 7400 1300 7400
+Connection ~ 1600 7100
 $EndSCHEMATC

Commit message: updates
Changed lines of the file:
@@
 Wire Wire Line
 	1600 7100 1800 7100
-Text Notes 850  5750 0    50   ~ 0
+Text Notes 700  6150 0    50   ~ 0
 Reset Circuit with digital select via p-mos select\n
 Wire Wire Line

Commit message: updates
Parts:
- added J?: Conn_02x03_Odd_Even, symbol Connector_Generic:Conn_02x03_Odd_Even
Connections:
- new net REQ_DTCE: J?.2 (Pin_2)
- new net REQ_HIZ: J?.4 (Pin_4)
- new net REQ_SHDN: J?.6 (Pin_6)
Other:
- moved on the sheet: C?, J?, Q?, R?, SW?, Y?
