File: Baseband.sch (KiCad schematic (older format))
At the start: 14 parts

Commit message: updates
Other:
- moved on the sheet: BZ?, C?, R?, RV?

Commit message: updates
Parts:
- C?: value C -> 100n
- R? (x2): value R -> 10K
Other:
- moved on the sheet: BZ?, C?, R?
Changed lines of the file:
@@
 Comment4 ""
 $EndDescr
-Text GLabel 4250 1550 0    50   Input ~ 0
+Text GLabel 4450 1550 0    50   Input ~ 0
 Baseband-IN
 Text GLabel 4250 4250 0    50   Output ~ 0
 Baseband-OUT
-Text GLabel 6000 1550 2    50   Output ~ 0
+Text GLabel 6200 1550 2    50   Output ~ 0
 Mega-PC0
 Text GLabel 6100 4000 2    50   Input ~ 0
 Mega-PB3
-Text GLabel 6100 5950 2    50   Input ~ 0
+Text GLabel 6100 6100 2    50   Input ~ 0
 Mega-PD3
 $Comp
 L Device:C_Polarized C?
 U 1 1 60EAC5FC
-P 4400 1550
+P 4600 1550
 AR Path="/60EAC5FC" Ref="C?"  Part="1"
 AR Path="/60EA1C1F/60EAC5FC" Ref="C?"  Part="1"
-F 0 "C?" V 4145 1550 50  0000 C CNN
-F 1 "3u3" V 4236 1550 50  0000 C CNN
-F 2 "" H 4438 1400 50  0001 C CNN
-F 3 "~" H 4400 1550 50  0001 C CNN
-	1    4400 1550
+F 0 "C?" V 4345 1550 50  0000 C CNN
+F 1 "3u3" V 4436 1550 50  0000 C CNN
+F 2 "" H 4638 1400 50  0001 C CNN
+F 3 "~" H 4600 1550 50  0001 C CNN
+	1    4600 1550
 	0    1    1    0
 $EndComp
@@
 L Device:R R?
 U 1 1 60EAC602
-P 4550 1700
+P 4900 1950
 AR Path="/60EAC602" Ref="R?"  Part="1"
 AR Path="/60EA1C1F/60EAC602" Ref="R?"  Part="1"
-F 0 "R?" H 4620 1746 50  0000 L CNN
-F 1 "10K" H 4620 1655 50  0000 L CNN
-F 2 "" V 4480 1700 50  0001 C CNN
-F 3 "~" H 4550 1700 50  0001 C CNN
-	1    4550 1700
+F 0 "R?" H 4970 1996 50  0000 L CNN
+F 1 "10K" H 4970 1905 50  0000 L CNN
+F 2 "" V 4830 1950 50  0001 C CNN
+F 3 "~" H 4900 1950 50  0001 C CNN
+	1    4900 1950
 	1    0    0    -1
 $EndComp
@@
 L Device:C C?
 U 1 1 60EAC608
-P 4550 2000
+P 4900 2400
 AR Path="/60EAC608" Ref="C?"  Part="1"
 AR Path="/60EA1C1F/60EAC608" Ref="C?"  Part="1"
-F 0 "C?" H 4665 2046 50  0000 L CNN
-F 1 "100n" H 4665 1955 50  0000 L CNN
-F 2 "" H 4588 1850 50  0001 C CNN
-F 3 "~" H 4550 2000 50  0001 C CNN
-	1    4550 2000
+F 0 "C?" H 5015 2446 50  0000 L CNN
+F 1 "100n" H 5015 2355 50  0000 L CNN
+F 2 "" H 4938 2250 50  0001 C CNN
+F 3 "~" H 4900 2400 50  0001 C CNN
+	1    4900 2400
 	1    0    0    -1
 $EndComp
@@
 L power:GND #PWR?
 U 1 1 60EAC60E
-P 4550 2150
+P 4900 2550
 AR Path="/60EAC60E" Ref="#PWR?"  Part="1"
 AR Path="/60EA1C1F/60EAC60E" Ref="#PWR?"  Part="1"
-F 0 "#PWR?" H 4550 1900 50  0001 C CNN
-F 1 "GND" H 4555 1977 50  0000 C CNN
-F 2 "" H 4550 2150 50  0001 C CNN
-F 3 "" H 4550 2150 50  0001 C CNN
-	1    4550 2150
+F 0 "#PWR?" H 4900 2300 50  0001 C CNN
+F 1 "GND" H 4905 2377 50  0000 C CNN
+F 2 "" H 4900 2550 50  0001 C CNN
+F 3 "" H 4900 2550 50  0001 C CNN
+	1    4900 2550
 	1    0    0    -1
 $EndComp
@@
 L power:GND #PWR?
 U 1 1 60EAC614
-P 5450 2650
+P 5450 2550
 AR Path="/60EAC614" Ref="#PWR?"  Part="1"
 AR Path="/60EA1C1F/60EAC614" Ref="#PWR?"  Part="1"
-F 0 "#PWR?" H 5450 2400 50  0001 C CNN
-F 1 "GND" H 5455 2477 50  0000 C CNN
-F 2 "" H 5450 2650 50  0001 C CNN
-F 3 "" H 5450 2650 50  0001 C CNN
-	1    5450 2650
+F 0 "#PWR?" H 5450 2300 50  0001 C CNN
+F 1 "GND" H 5455 2377 50  0000 C CNN
+F 2 "" H 5450 2550 50  0001 C CNN
+F 3 "" H 5450 2550 50  0001 C CNN
+	1    5450 2550
 	1    0    0    -1
 $EndComp
@@
 L Device:R R?
 U 1 1 60EAC61A
-P 5450 2500
+P 5450 2400
 AR Path="/60EAC61A" Ref="R?"  Part="1"
 AR Path="/60EA1C1F/60EAC61A" Ref="R?"  Part="1"
-F 0 "R?" H 5520 2546 50  0000 L CNN
-F 1 "R" H 5520 2455 50  0000 L CNN
-F 2 "" V 5380 2500 50  0001 C CNN
-F 3 "~" H 5450 2500 50  0001 C CNN
-	1    5450 2500
+F 0 "R?" H 5520 2446 50  0000 L CNN
+F 1 "10K" H 5520 2355 50  0000 L CNN
+F 2 "" V 5380 2400 50  0001 C CNN
+F 3 "~" H 5450 2400 50  0001 C CNN
+	1    5450 2400
 	1    0    0    -1
 $EndComp
@@
 L Device:R R?
 U 1 1 60EAC620
-P 5450 2200
+P 5450 1950
 AR Path="/60EAC620" Ref="R?"  Part="1"
 AR Path="/60EA1C1F/60EAC620" Ref="R?"  Part="1"
-F 0 "R?" H 5380 2154 50  0000 R CNN
-F 1 "R" H 5380 2245 50  0000 R CNN
-F 2 "" V 5380 2200 50  0001 C CNN
-F 3 "~" H 5450 2200 50  0001 C CNN
-	1    5450 2200
+F 0 "R?" H 5380 1904 50  0000 R CNN
+F 1 "10K" H 5380 1995 50  0000 R CNN
+F 2 "" V 5380 1950 50  0001 C CNN
+F 3 "~" H 5450 1950 50  0001 C CNN
+	1    5450 1950
 	-1   0    0    1
 $EndComp
-Wire Wire Line
-	5450 2350 4900 2350
-Connection ~ 4550 1550
 $Comp
 L Device:C C?
 U 1 1 60EAC628
-P 5800 2500
+P 6000 2400
 AR Path="/60EAC628" Ref="C?"  Part="1"
 AR Path="/60EA1C1F/60EAC628" Ref="C?"  Part="1"
-F 0 "C?" H 5915 2546 50  0000 L CNN
-F 1 "C" H 5915 2455 50  0000 L CNN
-F 2 "" H 5838 2350 50  0001 C CNN
-F 3 "~" H 5800 2500 50  0001 C CNN
-	1    5800 2500
+F 0 "C?" H 6115 2446 50  0000 L CNN
+F 1 "100n" H 6115 2355 50  0000 L CNN
+F 2 "" H 6038 2250 50  0001 C CNN
+F 3 "~" H 6000 2400 50  0001 C CNN
+	1    6000 2400
 	1    0    0    -1
 $EndComp
@@
 L power:GND #PWR?
 U 1 1 60EAC62E
-P 5800 2650
+P 6000 2550
 AR Path="/60EAC62E" Ref="#PWR?"  Part="1"
 AR Path="/60EA1C1F/60EAC62E" Ref="#PWR?"  Part="1"
-F 0 "#PWR?" H 5800 2400 50  0001 C CNN
-F 1 "GND" H 5805 2477 50  0000 C CNN
-F 2 "" H 5800 2650 50  0001 C CNN
-F 3 "" H 5800 2650 50  0001 C CNN
-	1    5800 2650
-	1    0    0    -1
-$EndComp
-Connection ~ 5450 2350
-Wire Wire Line
-	4550 1550 6000 1550
-Text GLabel 6000 2050 2    50   Output ~ 0
+F 0 "#PWR?" H 6000 2300 50  0001 C CNN
+F 1 "GND" H 6005 2377 50  0000 C CNN
+F 2 "" H 6000 2550 50  0001 C CNN
+F 3 "" H 6000 2550 50  0001 C CNN
+	1    6000 2550
+	1    0    0    -1
+$EndComp
+Text GLabel 6200 1700 2    50   Output ~ 0
 Mega-AREF
 Wire Wire Line
-	5450 2050 5800 2050
-Wire Wire Line
-	5800 2350 5800 2050
-Connection ~ 5800 2050
-Wire Wire Line
-	5800 2050 6000 2050
+	6000 2250 6000 1700
+Wire Wire Line
+	6000 1700 6200 1700
 $Comp
 L Device:Buzzer BZ?
 U 1 1 60EAC63B
-P 5100 6050
+P 5100 6000
 AR Path="/60EAC63B" Ref="BZ?"  Part="1"
 AR Path="/60EA1C1F/60EAC63B" Ref="BZ?"  Part="1"
-F 0 "BZ?" V 5058 6202 50  0000 L CNN
-F 1 "Buzzer" V 5149 6202 50  0000 L CNN
-F 2 "" V 5075 6150 50  0001 C CNN
-F 3 "~" V 5075 6150 50  0001 C CNN
-	1    5100 6050
-	0    1    1    0
+F 0 "BZ?" V 5058 6152 50  0000 L CNN
+F 1 "Buzzer" V 5149 6152 50  0000 L CNN
+F 2 "" V 5075 6100 50  0001 C CNN
+F 3 "~" V 5075 6100 50  0001 C CNN
+	1    5100 6000
+	0    1    -1   0
 $EndComp
 $Comp
 L Device:R R?
 U 1 1 60EAC641
-P 5650 5950
+P 5650 6100
 AR Path="/60EAC641" Ref="R?"  Part="1"
 AR Path="/60EA1C1F/60EAC641" Ref="R?"  Part="1"
-F 0 "R?" V 5443 5950 50  0000 C CNN
-F 1 "1K" V 5534 5950 50  0000 C CNN
-F 2 "" V 5580 5950 50  0001 C CNN
-F 3 "~" H 5650 5950 50  0001 C CNN
-	1    5650 5950
-	0    1    1    0
-$EndComp
-Wire Wire Line
-	5800 5950 6100 5950
-Wire Wire Line
-	5500 5950 5200 5950
-Wire Wire Line
-	5000 5950 4600 5950
+F 0 "R?" V 5443 6100 50  0000 C CNN
+F 1 "1K" V 5534 6100 50  0000 C CNN
+F 2 "" V 5580 6100 50  0001 C CNN
+F 3 "~" H 5650 6100 50  0001 C CNN
+	1    5650 6100
+	0    1    1    0
+$EndComp
+Wire Wire Line
+	5800 6100 6100 6100
+Wire Wire Line
+	5500 6100 5200 6100
+Wire Wire Line
+	5000 6100 4600 6100
 $Comp
 L power:GND #PWR?
 U 1 1 60EAC64A
-P 4600 5950
+P 4600 6100
 AR Path="/60EAC64A" Ref="#PWR?"  Part="1"
 AR Path="/60EA1C1F/60EAC64A" Ref="#PWR?"  Part="1"
-F 0 "#PWR?" H 4600 5700 50  0001 C CNN
-F 1 "GND" H 4605 5777 50  0000 C CNN
-F 2 "" H 4600 5950 50  0001 C CNN
-F 3 "" H 4600 5950 50  0001 C CNN
-	1    4600 5950
-	1    0    0    -1
+F 0 "#PWR?" H 4600 5850 50  0001 C CNN
+F 1 "GND" V 4600 5900 50  0000 C CNN
+F 2 "" H 4600 6100 50  0001 C CNN
+F 3 "" H 4600 6100 50  0001 C CNN
+	1    4600 6100
+	0    1    1    0
 $EndComp
 $Comp
@@
 Text Notes 5050 3450 0    50   ~ 0
 Baseband Output
-Text Notes 4700 5600 0    50   ~ 0
+Text Notes 4600 5600 0    50   ~ 0
 Baseband Monitor (via AT Command "M0/1")
 Wire Wire Line
-	4550 1850 4900 1850
-Connection ~ 4550 1850
-Wire Wire Line
-	4900 1850 4900 2350
-Wire Wire Line
 	4700 4400 4700 4450
+Wire Wire Line
+	4900 1800 4900 1550
+Wire Wire Line
+	4900 2100 4900 2150
+Wire Wire Line
+	4900 2150 5450 2150
+Connection ~ 4900 2150
+Wire Wire Line
+	4900 2150 4900 2250
+Wire Wire Line
+	5450 2100 5450 2150
+Connection ~ 5450 2150
+Wire Wire Line
+	5450 2150 5450 2250
+Wire Wire Line
+	4750 1550 4900 1550
+Connection ~ 4900 1550
+Wire Wire Line
+	4900 1550 6200 1550
+Wire Wire Line
+	6000 1700 5450 1700
+Wire Wire Line
+	5450 1700 5450 1800
+Connection ~ 6000 1700
 $EndSCHEMATC
